File: pcb/keyboard-x2-lumberjack-arm.kicad_pcb (KiCad board)
At the start: 2 copper layers, 285 x 94.2 mm, 146 parts, among them J1 16-pin USB-C Connector SMD, U1 STM32F103 Bluepill, or MiniF4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, U2 SN74LVC1T45DBV

Commit message: fix: replace pcb shape with svg shape
Other:
- outline, holes or cut-outs redrawn
- net class Default removed
- net class PWR removed

Commit message: fix: track too close to drilled hole
Parts:
- removed H5: ~, ProjectLocal:Bumpon_3M_F0502
- removed H6: ~, ProjectLocal:H_M2_Spacer_Hole
- removed HOLE (x2): Graphic_Mask_HalfHole, ProjectLocal:Graphic_Mask_HalfHole
- removed REF**: OSHW, lumberjack:OSHW
Connections:
- D4 pad 2: Net-(D4-Pad2) -> unconnected-(D4-Pad2)
- J1 pad A8: Net-(J1-PadA8) -> unconnected-(J1-PadA8)
- J1 pad B8: Net-(J1-PadB8) -> unconnected-(J1-PadB8)
- J1 pad S1: Net-(J1-PadS1) -> unconnected-(J1-PadS1)
- U1 pad 11: Net-(U1-Pad11) -> unconnected-(U1-Pad11)
- U1 pad 12: Net-(U1-Pad12) -> unconnected-(U1-Pad12)
- U1 pad 17: Net-(U1-Pad17) -> unconnected-(U1-Pad17)
- U1 pad 21: Net-(U1-Pad21) -> unconnected-(U1-Pad21)
- U1 pad 22: Net-(U1-Pad22) -> unconnected-(U1-Pad22)
- U1 pad 23: Net-(U1-Pad23) -> unconnected-(U1-Pad23)
- U1 pad 24: Net-(U1-Pad24) -> unconnected-(U1-Pad24)
- U1 pad 25: Net-(U1-Pad25) -> unconnected-(U1-Pad25)
- U1 pad 26: Net-(U1-Pad26) -> unconnected-(U1-Pad26)
- U1 pad 27: Net-(U1-Pad27) -> unconnected-(U1-Pad27)
- U1 pad 28: Net-(U1-Pad28) -> unconnected-(U1-Pad28)
- U1 pad 36: Net-(U1-Pad36) -> unconnected-(U1-Pad36)
- U1 pad 37: Net-(U1-Pad37) -> unconnected-(U1-Pad37)
- U1 pad 6: Net-(U1-Pad6) -> unconnected-(U1-Pad6)
Routing:
- net /COL7: track 135.7 -> 137.2 mm
- net /COL2: track 206.1 -> 206.8 mm
- net Net-(D_5_6-Pad2): track 55.0 -> 55.7 mm
