File: pcb/keyboard-x2-lumberjack-arm.kicad_pcb (KiCad board)
At the start: 2 copper layers, 285 x 94.2 mm, 141 parts, among them J1 16-pin USB-C Connector SMD, U1 STM32F103 Bluepill, or MiniF4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, U2 SN74LVC1T45DBV

Commit message: fix: track position
Routing:
- net Net-(D_3_6-Pad2): track 22.0 -> 23.3 mm
- net /COL7: track 136.2 -> 135.6 mm
- net /COL2: track 206.8 -> 206.2 mm

Commit message: fix: update gh60 mounting hole footprint
Parts:
- added H5: ~, Lumberjack:MountingSlot_M2, F.Cu at (43.2, 106.5)
- added H6: ~, Lumberjack:MountingSlot_M2, F.Cu at (342.9, 106.5)
- H7: footprint ProjectLocal:H_M2_Spacer_Hole -> Lumberjack:MountingSlot_M2

Commit message: fix: update board setup constraint to match Lumberjack's
Parts:
- moved H6 7.89 mm to (335.0, 106.5)
- moved H5 6.83 mm to (50.0, 106.5)
Other:
- outline, holes or cut-outs redrawn
