File: pcb/demo-usb-16pin.kicad_pcb (KiCad board)
At the start: 2 copper layers, 40.2 x 23.6 mm, 7 parts, among them J1 USB_C_Receptacle_USB2.0, J2 Conn_01x04_Female, J3 Conn_01x04_Female, J4 Conn_01x10_Female

Commit message: pcb: demo-usb-16pin: update to kicad 6
Other:
- net class Default removed
- net class Power removed
