File: pcb/demo-usb-16pin.kicad_pcb (KiCad board)
At the start: 2 copper layers, 40.2 x 23.6 mm, 7 parts, among them J1 USB_C_Receptacle_USB2.0, J2 Conn_01x04_Female, J3 Conn_01x04_Female, J4 Conn_01x10_Female

Commit message: pcb: tidy values in demo-usb-16pin
Parts:
- J1: value USB_C_Receptacle_USB2.0 -> USB Type-C Female 16P
- R1, R2: value 5.1K -> 5.1k
