File: pcb/keyboard-x2-switch-matrix.kicad_sch (KiCad schematic)
At the start: 120 parts

Commit message: pcb: x-2 hsrgb: fix values/descriptions (for ibom)
Parts:
- SW_1_1, SW_1_10, SW_1_11, SW_1_12, SW_1_2, SW_1_3, SW_1_4, SW_1_5, SW_1_6, SW_1_7, SW_1_8, SW_1_9, SW_2_1, SW_2_10, SW_2_11, SW_2_12, SW_2_2, SW_2_3, SW_2_4, SW_2_5, SW_2_6, SW_2_7, SW_2_8, SW_2_9, SW_3_1, SW_3_10, SW_3_11, SW_3_12, SW_3_2, SW_3_3, SW_3_4, SW_3_5, SW_3_6, SW_3_7, SW_3_8, SW_3_9, SW_4_1, SW_4_10, SW_4_11, SW_4_12, SW_4_2, SW_4_3, SW_4_4, SW_4_5, SW_4_6, SW_4_7, SW_4_8, SW_4_9, SW_5_1, SW_5_10, SW_5_11, SW_5_12, SW_5_2, SW_5_3, SW_5_4, SW_5_5, SW_5_6, SW_5_7, SW_5_8, SW_5_9: value MX-compatible or Kailh Choc v1 -> Kailh MX hotswap socket
