File: pcb/keyboard-pico42.kicad_pcb (KiCad board)
At the start: 2 copper layers, 224.6 x 72.2 mm, 95 parts, among them U1 Pico

Commit message: pcb: update user comments in keyboard-pico42
Other:
- board text added: "PCB outline generated with pico42_pcb_outline.scad. Positions of most components managed Kicad scripting console, with source in scripts/kicad_helpers."
Changed lines of the file:
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@@
     (effects (font (size 0.8 0.8) (thickness 0.16)) (justify mirror))
+  )
+  (gr_text "PCB outline generated with pico42_pcb_outline.scad.\n\nPositions of most components managed Kicad scripting\nconsole, with source in scripts/kicad_helpers." (at 52.578 152.1206) (layer "Cmts.User")
+    (effects (font (size 4 4) (thickness 0.15)) (justify left bottom))
   )
   (target plus (at 57.5 57.5) (size 5) (width 0.09906) (layer "Edge.Cuts"))
