File: pcb/keyboard-ch552-44.kicad_pcb (KiCad board)
At the start: 2 copper layers, 224.6 x 74.2 mm, 101 parts, among them J1 USB_C_Receptacle_USB2.0, U1 WeAct_CH552CoreBoard

Commit message: pcb: CH552-44: update more fields
Parts:
- H1, H10, H2, H3, H4, H5, H7, H8, H9: value MountingHole -> M2 screw
- J1: value USB_C_Receptacle_USB2.0 -> 16-pin USB-C Connector SMD
- SW_1_1, SW_1_2, SW_1_3, SW_1_5, SW_1_6, SW_1_7, SW_2_1, SW_2_2, SW_2_3, SW_2_4, SW_2_5, SW_2_6, SW_2_7, SW_3_1, SW_3_2, SW_3_3, SW_3_4, SW_3_5, SW_3_6, SW_3_7, SW_4_1, SW_4_2, SW_4_3, SW_4_5, SW_4_6, SW_4_7, SW_5_1, SW_5_2, SW_5_3, SW_5_5, SW_5_6, SW_5_7, SW_6_1, SW_6_2, SW_6_3, SW_6_4, SW_6_5, SW_6_6, SW_6_7, SW_7_1, SW_7_2, SW_7_4, SW_7_5, SW_7_6: value MX-compatible or Kailh Choc v1 -> MX-compatible

Commit message: pcb: update user comments in keyboard-ch552-44
Other:
- board text added: "PCB outline generated with pico42_pcb_outline.scad. Positions of most components managed Kicad scripting console, with source in scripts/kicad_helpers."
Changed lines of the file:
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@@
     (effects (font (size 0.8 0.8) (thickness 0.16)) (justify mirror))
+  )
+  (gr_text "PCB outline generated with pico42_pcb_outline.scad.\n\nPositions of most components managed Kicad scripting\nconsole, with source in scripts/kicad_helpers." (at 51.943 150.8506) (layer "Cmts.User")
+    (effects (font (size 4 4) (thickness 0.15)) (justify left bottom))
   )
   (target plus (at 57.5 57.5) (size 5) (width 0.09906) (layer "Edge.Cuts"))
