File: pcb/keyboard-ch552-48.kicad_pcb (KiCad board)
At the start: 2 copper layers, 224.6 x 74.2 mm, 112 parts, among them J1 USB_C_Receptacle_USB2.0, SW1 SW_SPST, SW2 SW_SPST, U1 WeAct_CH552CoreBoard

Commit message: pcb: update user comments in keyboard-ch552-48
Other:
- board text added: "PCB outline generated with pico42_pcb_outline.scad. Positions of most components managed Kicad scripting console, with source in scripts/kicad_helpers."
Changed lines of the file:
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@@
     (effects (font (size 1 1) (thickness 0.15)) (justify left bottom mirror))
+  )
+  (gr_text "PCB outline generated with pico42_pcb_outline.scad.\n\nPositions of most components managed Kicad scripting\nconsole, with source in scripts/kicad_helpers." (at 52.0446 149.8092) (layer "Cmts.User")
+    (effects (font (size 4 4) (thickness 0.15)) (justify left bottom))
   )
   (target plus (at 57.5 57.5) (size 5) (width 0.09906) (layer "Edge.Cuts"))
