File: pcb/keyboard-pykey40-lite.kicad_pcb (KiCad board)
At the start: 2 copper layers, 227 x 77 mm, 136 parts, among them J1 USB_C_Receptacle_USB2.0, J2 Conn_01x03, U1 RP2040, U2 W25Q128JVS, U3 USBLC6-2SC6, U4 AMS1117-3.3, Y1 12MHz

Commit message: pcb: update user comments in keyboard-pykey40-lite
Other:
- board text added: "PCB outline generated with jj40_pcb_outline.scad."
Changed lines of the file:
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@@
     (effects (font (size 1.524 1.524) (thickness 0.3048)))
+  )
+  (gr_text "PCB outline generated with jj40_pcb_outline.scad." (at 53.086 134.3914) (layer "Cmts.User")
+    (effects (font (size 4 4) (thickness 0.15)) (justify left bottom))
   )
   (target plus (at 57.5 58.5) (size 5) (width 0.09906) (layer "Edge.Cuts"))
