File: pcb/keyboard-pykey40-lite.kicad_pcb (KiCad board)
At the start: 2 copper layers, 227 x 77 mm, 136 parts, among them J1 USB_C_Receptacle_USB2.0, J2 Conn_01x03, U1 RP2040, U2 W25Q128JVS, U3 USBLC6-2SC6, U4 AMS1117-3.3, Y1 12MHz

Commit message: pcb: tidy values in pykey40-lite
Parts:
- C1, C14, C2, C3, C4, C5, C6, C7, C8, C9: value 100n -> 100nF
- C10, C11: value 1u -> 1uF
- C12, C13: value 22p -> 22pF
- C15, C16: value 22u -> 22uF
- J1: value USB_C_Receptacle_USB2.0 -> USB Type-C Female 16P
- R3, R4: value 22 -> 22R
