File: pcb/keyboard-ch32x-48.kicad_pcb (KiCad board)
At the start: 2 copper layers, 224.6 x 74.2 mm, 117 parts, among them J1 USB_C_Receptacle_USB2.0, J2 Conn_01x02, J3 Conn_01x04, SW1 SW_SPST, SW2 SW_SPST, U1 CH32X033F8P6

Commit message: pcb: ch32x-48 rev 2025.2
Parts:
- removed D_5_1, D_5_2, D_5_3, D_5_4, D_5_5, D_5_6, D_5_7, D_6_1, D_6_2, D_6_3, D_6_4, D_6_5, D_6_6, D_6_7, D_7_1, D_7_2, D_7_3, D_7_4, D_7_5, D_7_6: 1N4148, Diode_SMD:D_1206_3216Metric
- removed SW_5_1, SW_5_2, SW_5_3, SW_5_4, SW_5_5, SW_5_6, SW_5_7, SW_6_1, SW_6_2, SW_6_3, SW_6_4, SW_6_5, SW_6_6, SW_6_7, SW_7_1, SW_7_2, SW_7_3, SW_7_4, SW_7_5, SW_7_6: MX-compatible, ProjectLocal:SW_Cherry_MX_PCB_1.00u_BSilkRef
- added D_1_10: 1N4148, Diode_SMD:D_1206_3216Metric, B.Cu at (220.9, 57.5)
- added D_1_11: 1N4148, Diode_SMD:D_1206_3216Metric, B.Cu at (256.0, 57.5)
- added D_1_12: 1N4148, Diode_SMD:D_1206_3216Metric, B.Cu at (259.0, 57.5)
- added D_1_8: 1N4148, Diode_SMD:D_1206_3216Metric, B.Cu at (182.8, 57.5)
- added D_1_9: 1N4148, Diode_SMD:D_1206_3216Metric, B.Cu at (217.9, 57.5)
- added D_2_10: 1N4148, Diode_SMD:D_1206_3216Metric, B.Cu at (220.9, 76.5)
- added D_2_11: 1N4148, Diode_SMD:D_1206_3216Metric, B.Cu at (256.0, 76.5)
- added D_2_12: 1N4148, Diode_SMD:D_1206_3216Metric, B.Cu at (259.0, 76.5)
- added D_2_8: 1N4148, Diode_SMD:D_1206_3216Metric, B.Cu at (182.8, 76.5)
- added D_2_9: 1N4148, Diode_SMD:D_1206_3216Metric, B.Cu at (217.9, 76.5)
- added D_3_10: 1N4148, Diode_SMD:D_1206_3216Metric, B.Cu at (220.9, 95.6)
- added D_3_11: 1N4148, Diode_SMD:D_1206_3216Metric, B.Cu at (256.0, 95.6)
- added D_3_12: 1N4148, Diode_SMD:D_1206_3216Metric, B.Cu at (259.0, 95.6)
- added D_3_8: 1N4148, Diode_SMD:D_1206_3216Metric, B.Cu at (182.8, 95.6)
- added D_3_9: 1N4148, Diode_SMD:D_1206_3216Metric, B.Cu at (217.9, 95.6)
- added D_4_10: 1N4148, Diode_SMD:D_1206_3216Metric, B.Cu at (220.9, 114.7)
- added D_4_11: 1N4148, Diode_SMD:D_1206_3216Metric, B.Cu at (256.0, 114.7)
- added D_4_12: 1N4148, Diode_SMD:D_1206_3216Metric, B.Cu at (259.0, 114.7)
- added D_4_8: 1N4148, Diode_SMD:D_1206_3216Metric, B.Cu at (182.8, 114.7)
- added D_4_9: 1N4148, Diode_SMD:D_1206_3216Metric, B.Cu at (217.9, 114.7)
- added SW_1_10: Redragon Low Profile switches, Switch_Keyboard_Cherry_MX:SW_Cherry_MX_PCB_1.00u, F.Cu at (228.9, 57.5)
- added SW_1_11: Redragon Low Profile switches, Switch_Keyboard_Cherry_MX:SW_Cherry_MX_PCB_1.00u, F.Cu at (248.0, 57.5)
- added SW_1_12: Redragon Low Profile switches, Switch_Keyboard_Cherry_MX:SW_Cherry_MX_PCB_1.00u, F.Cu at (267.1, 57.5)
- added SW_1_8: Redragon Low Profile switches, Switch_Keyboard_Cherry_MX:SW_Cherry_MX_PCB_1.00u, F.Cu at (190.8, 57.5)
- added SW_1_9: Redragon Low Profile switches, Switch_Keyboard_Cherry_MX:SW_Cherry_MX_PCB_1.00u, F.Cu at (209.9, 57.5)
- added SW_2_10: Redragon Low Profile switches, Switch_Keyboard_Cherry_MX:SW_Cherry_MX_PCB_1.00u, F.Cu at (228.9, 76.5)
- added SW_2_11: Redragon Low Profile switches, Switch_Keyboard_Cherry_MX:SW_Cherry_MX_PCB_1.00u, F.Cu at (248.0, 76.5)
- added SW_2_12: Redragon Low Profile switches, Switch_Keyboard_Cherry_MX:SW_Cherry_MX_PCB_1.00u, F.Cu at (267.1, 76.5)
- added SW_2_8: Redragon Low Profile switches, Switch_Keyboard_Cherry_MX:SW_Cherry_MX_PCB_1.00u, F.Cu at (190.8, 76.5)
- added SW_2_9: Redragon Low Profile switches, Switch_Keyboard_Cherry_MX:SW_Cherry_MX_PCB_1.00u, F.Cu at (209.9, 76.5)
- added SW_3_10: Redragon Low Profile switches, Switch_Keyboard_Cherry_MX:SW_Cherry_MX_PCB_1.00u, F.Cu at (228.9, 95.6)
- added SW_3_11: Redragon Low Profile switches, Switch_Keyboard_Cherry_MX:SW_Cherry_MX_PCB_1.00u, F.Cu at (248.0, 95.6)
- added SW_3_12: Redragon Low Profile switches, Switch_Keyboard_Cherry_MX:SW_Cherry_MX_PCB_1.00u, F.Cu at (267.1, 95.6)
- added SW_3_8: Redragon Low Profile switches, Switch_Keyboard_Cherry_MX:SW_Cherry_MX_PCB_1.00u, F.Cu at (190.8, 95.6)
- added SW_3_9: Redragon Low Profile switches, Switch_Keyboard_Cherry_MX:SW_Cherry_MX_PCB_1.00u, F.Cu at (209.9, 95.6)
- added SW_4_10: Redragon Low Profile switches, Switch_Keyboard_Cherry_MX:SW_Cherry_MX_PCB_1.00u, F.Cu at (228.9, 114.7)
- added SW_4_11: Redragon Low Profile switches, Switch_Keyboard_Cherry_MX:SW_Cherry_MX_PCB_1.00u, F.Cu at (248.0, 114.7)
- added SW_4_12: Redragon Low Profile switches, Switch_Keyboard_Cherry_MX:SW_Cherry_MX_PCB_1.00u, F.Cu at (267.1, 114.7)
- added SW_4_8: Redragon Low Profile switches, Switch_Keyboard_Cherry_MX:SW_Cherry_MX_PCB_1.00u, F.Cu at (190.8, 114.7)
- added SW_4_9: Redragon Low Profile switches, Switch_Keyboard_Cherry_MX:SW_Cherry_MX_PCB_1.00u, F.Cu at (209.9, 114.7)
- SW_1_1, SW_1_2, SW_1_3, SW_1_4, SW_1_5, SW_1_6, SW_1_7, SW_2_1, SW_2_2, SW_2_3, SW_2_4, SW_2_5, SW_2_6, SW_2_7, SW_3_1, SW_3_2, SW_3_3, SW_3_4, SW_3_5, SW_3_6, SW_3_7, SW_4_1, SW_4_2, SW_4_3, SW_4_4, SW_4_5, SW_4_6, SW_4_7: value MX-compatible -> Redragon Low Profile switches; footprint ProjectLocal:SW_Cherry_MX_PCB_1.00u_BSilkRef -> Switch_Keyboard_Cherry_MX:SW_Cherry_MX_PCB_1.00u
- U1: value CH32X033F8P6 -> CH32X035C8T6; footprint Package_SO:TSSOP-20_4.4x6.5mm_P0.65mm -> Package_QFP:LQFP-48_7x7mm_P0.5mm
- moved H2 194.3 mm to (257.5, 67.0)
- moved H4 194.3 mm to (67.0, 105.1)
- moved SW_4_7 102.6 mm to (171.8, 114.7)
- moved SW_3_7 102.6 mm to (171.8, 95.6)
- moved H3 97.1 mm to (162.3, 86.1)
- moved H5 97.1 mm to (257.5, 105.1)
- moved D_1_6 92.9 mm to (144.7, 57.5), turned to 90 degrees
- moved D_4_4 92.9 mm to (106.6, 114.7), turned to 90 degrees
- moved D_3_7 87.9 mm to (179.8, 95.6), turned to 90 degrees
- moved D_4_7 87.9 mm to (179.8, 114.7), turned to 90 degrees
- moved D_1_7 85.2 mm to (179.8, 57.5), turned to 90 degrees
- moved D_2_7 85.2 mm to (179.8, 76.5), turned to 90 degrees
- moved SW_1_7 85.2 mm to (171.8, 57.5)
- moved SW_2_7 85.2 mm to (171.8, 76.5)
- moved SW_1_6 80.8 mm to (152.8, 57.5)
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Connections:
- D_1_1 pad 1: Net-(D_1_1-K) -> /ROW1
- D_1_1 pad 2: /ROW1 -> Net-(D_1_1-A)
- D_1_2 pad 1: Net-(D_1_2-K) -> /ROW1
- D_1_2 pad 2: /ROW1 -> Net-(D_1_2-A)
- D_1_3 pad 1: Net-(D_1_3-K) -> /ROW1
- D_1_3 pad 2: /ROW1 -> Net-(D_1_3-A)
- D_1_4 pad 1: Net-(D_1_4-K) -> /ROW1
- D_1_4 pad 2: /ROW1 -> Net-(D_1_4-A)
- D_1_5 pad 1: Net-(D_1_5-K) -> /ROW1
- D_1_5 pad 2: /ROW1 -> Net-(D_1_5-A)
- D_1_6 pad 1: Net-(D_1_6-K) -> /ROW1
- D_1_6 pad 2: /ROW1 -> Net-(D_1_6-A)
- D_1_7 pad 1: Net-(D_1_7-K) -> /ROW1
- D_1_7 pad 2: /ROW1 -> Net-(D_1_7-A)
- D_2_1 pad 1: Net-(D_2_1-K) -> /ROW2
- D_2_1 pad 2: /DCK -> Net-(D_2_1-A)
- D_2_2 pad 1: Net-(D_2_2-K) -> /ROW2
- D_2_2 pad 2: /DCK -> Net-(D_2_2-A)
- D_2_3 pad 1: Net-(D_2_3-K) -> /ROW2
- D_2_3 pad 2: /DCK -> Net-(D_2_3-A)
- D_2_4 pad 1: Net-(D_2_4-K) -> /ROW2
- D_2_4 pad 2: /DCK -> Net-(D_2_4-A)
- D_2_5 pad 1: Net-(D_2_5-K) -> /ROW2
- D_2_5 pad 2: /DCK -> Net-(D_2_5-A)
- D_2_6 pad 1: Net-(D_2_6-K) -> /ROW2
- D_2_6 pad 2: /DCK -> Net-(D_2_6-A)
- D_2_7 pad 1: Net-(D_2_7-K) -> /ROW2
- D_2_7 pad 2: /DCK -> Net-(D_2_7-A)
- D_3_1 pad 1: Net-(D_3_1-K) -> /ROW3
- D_3_1 pad 2: /ROW3 -> Net-(D_3_1-A)
- D_3_2 pad 1: Net-(D_3_2-K) -> /ROW3
- D_3_2 pad 2: /ROW3 -> Net-(D_3_2-A)
- D_3_3 pad 1: Net-(D_3_3-K) -> /ROW3
- D_3_3 pad 2: /ROW3 -> Net-(D_3_3-A)
- D_3_4 pad 1: Net-(D_3_4-K) -> /ROW3
- D_3_4 pad 2: /ROW3 -> Net-(D_3_4-A)
- D_3_5 pad 1: Net-(D_3_5-K) -> /ROW3
- D_3_5 pad 2: /ROW3 -> Net-(D_3_5-A)
- D_3_6 pad 1: Net-(D_3_6-K) -> /ROW3
- D_3_6 pad 2: /ROW3 -> Net-(D_3_6-A)
- D_3_7 pad 1: Net-(D_3_7-K) -> /ROW3
- D_3_7 pad 2: /ROW3 -> Net-(D_3_7-A)
- D_4_1 pad 1: Net-(D_4_1-K) -> /ROW4
- D_4_1 pad 2: /ROW4 -> Net-(D_4_1-A)
- D_4_2 pad 1: Net-(D_4_2-K) -> /ROW4
- D_4_2 pad 2: /ROW4 -> Net-(D_4_2-A)
- D_4_3 pad 1: Net-(D_4_3-K) -> /ROW4
- D_4_3 pad 2: /ROW4 -> Net-(D_4_3-A)
- D_4_4 pad 1: Net-(D_4_4-K) -> /ROW4
- D_4_4 pad 2: /ROW4 -> Net-(D_4_4-A)
- D_4_5 pad 1: Net-(D_4_5-K) -> /ROW4
- D_4_5 pad 2: /ROW4 -> Net-(D_4_5-A)
- D_4_6 pad 1: Net-(D_4_6-K) -> /ROW4
- D_4_6 pad 2: /ROW4 -> Net-(D_4_6-A)
- D_4_7 pad 1: Net-(D_4_7-K) -> /ROW4
- D_4_7 pad 2: /ROW4 -> Net-(D_4_7-A)
- J2 pad 1: /ROW4 -> /TX
- J2 pad 2: /ROW3 -> /RX
- SW_1_1 pad 2: Net-(D_1_1-K) -> Net-(D_1_1-A)
- SW_1_2 pad 2: Net-(D_1_2-K) -> Net-(D_1_2-A)
- SW_1_3 pad 2: Net-(D_1_3-K) -> Net-(D_1_3-A)
- SW_1_4 pad 2: Net-(D_1_4-K) -> Net-(D_1_4-A)
- SW_1_5 pad 2: Net-(D_1_5-K) -> Net-(D_1_5-A)
- SW_1_6 pad 2: Net-(D_1_6-K) -> Net-(D_1_6-A)
- SW_1_7 pad 2: Net-(D_1_7-K) -> Net-(D_1_7-A)
- SW_2_1 pad 2: Net-(D_2_1-K) -> Net-(D_2_1-A)
- SW_2_2 pad 2: Net-(D_2_2-K) -> Net-(D_2_2-A)
- SW_2_3 pad 2: Net-(D_2_3-K) -> Net-(D_2_3-A)
- SW_2_4 pad 2: Net-(D_2_4-K) -> Net-(D_2_4-A)
- SW_2_5 pad 2: Net-(D_2_5-K) -> Net-(D_2_5-A)
- SW_2_6 pad 2: Net-(D_2_6-K) -> Net-(D_2_6-A)
- SW_2_7 pad 2: Net-(D_2_7-K) -> Net-(D_2_7-A)
- SW_3_1 pad 2: Net-(D_3_1-K) -> Net-(D_3_1-A)
- SW_3_2 pad 2: Net-(D_3_2-K) -> Net-(D_3_2-A)
- SW_3_3 pad 2: Net-(D_3_3-K) -> Net-(D_3_3-A)
- SW_3_4 pad 2: Net-(D_3_4-K) -> Net-(D_3_4-A)
- SW_3_5 pad 2: Net-(D_3_5-K) -> Net-(D_3_5-A)
- SW_3_6 pad 2: Net-(D_3_6-K) -> Net-(D_3_6-A)
- SW_3_7 pad 2: Net-(D_3_7-K) -> Net-(D_3_7-A)
- SW_4_1 pad 2: Net-(D_4_1-K) -> Net-(D_4_1-A)
- SW_4_2 pad 2: Net-(D_4_2-K) -> Net-(D_4_2-A)
- SW_4_3 pad 2: Net-(D_4_3-K) -> Net-(D_4_3-A)
- SW_4_4 pad 2: Net-(D_4_4-K) -> Net-(D_4_4-A)
- SW_4_5 pad 2: Net-(D_4_5-K) -> Net-(D_4_5-A)
- SW_4_6 pad 2: Net-(D_4_6-K) -> Net-(D_4_6-A)
- SW_4_7 pad 2: Net-(D_4_7-K) -> Net-(D_4_7-A)
- U1 pad 1: /COL2 -> /TX
- U1 pad 10: /COL3 -> unconnected-(U1-PA0-Pad10)
- U1 pad 11: /COL7 -> unconnected-(U1-PA1-Pad11)
- U1 pad 12: /COL6 -> /ROW2
- U1 pad 13: /COL5 -> unconnected-(U1-PA3-Pad13)
- U1 pad 14: /COL4 -> /ROW3
- U1 pad 15: /ROW5 -> unconnected-(U1-PA5-Pad15)
- U1 pad 17: /ROW3 -> unconnected-(U1-PA7-Pad17)
- U1 pad 18: /DCK -> unconnected-(U1-PC6-Pad18)
- U1 pad 19: /ROW1 -> unconnected-(U1-PC7-Pad19)
- U1 pad 2: /ROW7 -> /RX
- U1 pad 20: /LED -> unconnected-(U1-PB0-Pad20)
- U1 pad 3: /COL1 -> /COL12
- U1 pad 4: /RESET -> /COL11
- U1 pad 5: /DM -> /COL10
- U1 pad 6: /DOWNLOAD -> /COL9
- U1 pad 7: /GND -> /RESET
- U1 pad 8: /DIO -> /COL8
- U1 pad 9: /VDD -> /COL7
Routing:
- net /DIO: track 488.5 -> 18.7 mm, vias 28 -> 4
- net /ROW7: track 426.4 -> 0.00 mm, vias 20 -> 0
- net /DCK: track 427.7 -> 12.8 mm, vias 26 -> 2
- net /ROW5: track 406.6 -> 0.00 mm, vias 16 -> 0
- net /ROW2: track 0.00 -> 207.2 mm
- net /ROW1: track 409.3 -> 217.9 mm, vias 20 -> 8
- net /ROW3: track 406.0 -> 224.4 mm, vias 20 -> 2
- net /COL12: track 0.00 -> 154.0 mm, vias 0 -> 3
- net /ROW4: track 383.1 -> 244.3 mm, vias 12 -> 4
- net /COL11: track 0.00 -> 135.3 mm, vias 0 -> 8
- net /COL7: track 195.0 -> 62.4 mm, vias 5 -> 6
- net /COL10: track 0.00 -> 116.6 mm, vias 0 -> 11
- net /COL6: track 180.6 -> 66.7 mm, vias 10 -> 9
- net /COL9: track 0.00 -> 97.1 mm, vias 0 -> 8
- net /COL8: track 0.00 -> 78.3 mm, vias 0 -> 11
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- added copper zone on B.Cu, net /GND
- added copper zone on F.Cu, net /GND
