File: pcb/keyboard-ch32x-48.kicad_pcb (KiCad board)
At the start: 2 copper layers, 224.6 x 74.2 mm, 117 parts, among them J1 USB_C_Receptacle_USB2.0, J2 Conn_01x02, J3 Conn_01x04, SW1 SW_SPST, SW2 SW_SPST, U1 CH32X035C8T6

Commit message: pcb: CH32X-48: fix incorrect value for SW_r_c
Parts:
- SW_1_1, SW_1_10, SW_1_11, SW_1_12, SW_1_2, SW_1_3, SW_1_4, SW_1_5, SW_1_6, SW_1_7, SW_1_8, SW_1_9, SW_2_1, SW_2_10, SW_2_11, SW_2_12, SW_2_2, SW_2_3, SW_2_4, SW_2_5, SW_2_6, SW_2_7, SW_2_8, SW_2_9, SW_3_1, SW_3_10, SW_3_11, SW_3_12, SW_3_2, SW_3_3, SW_3_4, SW_3_5, SW_3_6, SW_3_7, SW_3_8, SW_3_9, SW_4_1, SW_4_10, SW_4_11, SW_4_12, SW_4_2, SW_4_3, SW_4_4, SW_4_5, SW_4_6, SW_4_7, SW_4_8, SW_4_9: value Redragon Low Profile switches -> MX-compatible
Changed lines of the file:
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@@
 			)
 		)
-		(property "Value" "Redragon Low Profile switches"
+		(property "Value" "MX-compatible"
 			(at 0 8 0)
 			(layer "F.Fab")
@@
 			)
 		)
-		(property "Value" "Redragon Low Profile switches"
+		(property "Value" "MX-compatible"
 			(at 0 8 0)
 			(layer "F.Fab")
@@
 			)
 		)
-		(property "Value" "Redragon Low Profile switches"
+		(property "Value" "MX-compatible"
 			(at 0 8 0)
 			(layer "F.Fab")
@@
 			)
 		)
-		(property "Value" "Redragon Low Profile switches"
+		(property "Value" "MX-compatible"
 			(at 0 8 0)
 			(layer "F.Fab")
@@
 			)
 		)
-		(property "Value" "Redragon Low Profile switches"
+		(property "Value" "MX-compatible"
 			(at 0 8 0)
 			(layer "F.Fab")
@@
 			)
 		)
-		(property "Value" "Redragon Low Profile switches"
+		(property "Value" "MX-compatible"
 			(at 0 8 0)
 			(layer "F.Fab")
@@
 			)
 		)
-		(property "Value" "Redragon Low Profile switches"
+		(property "Value" "MX-compatible"
 			(at 0 8 0)
 			(layer "F.Fab")
@@
 			)
 		)
-		(property "Value" "Redragon Low Profile switches"
+		(property "Value" "MX-compatible"
 			(at 0 8 0)
 			(layer "F.Fab")
@@
 			)
 		)
-		(property "Value" "Redragon Low Profile switches"
+		(property "Value" "MX-compatible"
 			(at 0 8 0)
 			(layer "F.Fab")
@@
 			)
 		)
-		(property "Value" "Redragon Low Profile switches"
+		(property "Value" "MX-compatible"
 			(at 0 8 0)
 			(layer "F.Fab")
@@
 			)
 		)
-		(property "Value" "Redragon Low Profile switches"
+		(property "Value" "MX-compatible"
 			(at 0 8 0)
 			(layer "F.Fab")
@@
 			)
 		)
-		(property "Value" "Redragon Low Profile switches"
+		(property "Value" "MX-compatible"
 			(at 0 8 0)
 			(layer "F.Fab")
@@
 			)
 		)
-		(property "Value" "Redragon Low Profile switches"
+		(property "Value" "MX-compatible"
 			(at 0 8 0)
 			(layer "F.Fab")
@@
 			)
 		)
-		(property "Value" "Redragon Low Profile switches"
+		(property "Value" "MX-compatible"
 			(at 0 8 0)
 			(layer "F.Fab")
@@
 			)
 		)
-		(property "Value" "Redragon Low Profile switches"
+		(property "Value" "MX-compatible"
 			(at 0 8 0)
 			(layer "F.Fab")
@@
 			)
 		)
-		(property "Value" "Redragon Low Profile switches"
+		(property "Value" "MX-compatible"
 			(at 0 8 0)
 			(layer "F.Fab")
@@
 			)
 		)
-		(property "Value" "Redragon Low Profile switches"
+		(property "Value" "MX-compatible"
 			(at 0 8 0)
 			(layer "F.Fab")
@@
 			)
 		)
-		(property "Value" "Redragon Low Profile switches"
+		(property "Value" "MX-compatible"
 			(at 0 8 0)
 			(layer "F.Fab")
@@
 			)
 		)
-		(property "Value" "Redragon Low Profile switches"
+		(property "Value" "MX-compatible"
 			(at 0 8 0)
 			(layer "F.Fab")
@@
 			)
 		)
-		(property "Value" "Redragon Low Profile switches"
+		(property "Value" "MX-compatible"
 			(at 0 8 0)
 			(layer "F.Fab")
@@
 			)
 		)
-		(property "Value" "Redragon Low Profile switches"
+		(property "Value" "MX-compatible"
 			(at 0 8 0)
 			(layer "F.Fab")
@@
 			)
 		)
-		(property "Value" "Redragon Low Profile switches"
+		(property "Value" "MX-compatible"
 			(at 0 8 0)
 			(layer "F.Fab")
@@
 			)
 		)
-		(property "Value" "Redragon Low Profile switches"
+		(property "Value" "MX-compatible"
 			(at 0 8 0)
 			(layer "F.Fab")
@@
 			)
 		)
-		(property "Value" "Redragon Low Profile switches"
+		(property "Value" "MX-compatible"
 			(at 0 8 0)
 			(layer "F.Fab")
@@
 			)
 		)
-		(property "Value" "Redragon Low Profile switches"
+		(property "Value" "MX-compatible"
 			(at 0 8 0)
 			(layer "F.Fab")
@@
 			)
 		)
-		(property "Value" "Redragon Low Profile switches"
+		(property "Value" "MX-compatible"
 			(at 0 8 0)
 			(layer "F.Fab")
@@
 			)
 		)
-		(property "Value" "Redragon Low Profile switches"
+		(property "Value" "MX-compatible"
 			(at 0 8 0)
 			(layer "F.Fab")
@@
 			)
 		)
-		(property "Value" "Redragon Low Profile switches"
+		(property "Value" "MX-compatible"
 			(at 0 8 0)
 			(layer "F.Fab")
@@
 			)
 		)
-		(property "Value" "Redragon Low Profile switches"
+		(property "Value" "MX-compatible"
 			(at 0 8 0)
 			(layer "F.Fab")
@@
 			)
 		)
-		(property "Value" "Redragon Low Profile switches"
+		(property "Value" "MX-compatible"
 			(at 0 8 0)
 			(layer "F.Fab")
@@
 			)
 		)
-		(property "Value" "Redragon Low Profile switches"
+		(property "Value" "MX-compatible"
 			(at 0 8 0)
 			(layer "F.Fab")
@@
 			)
 		)
-		(property "Value" "Redragon Low Profile switches"
+		(property "Value" "MX-compatible"
 			(at 0 8 0)
 			(layer "F.Fab")
@@
 			)
 		)
-		(property "Value" "Redragon Low Profile switches"
+		(property "Value" "MX-compatible"
 			(at 0 8 0)
 			(layer "F.Fab")
@@
 			)
 		)
-		(property "Value" "Redragon Low Profile switches"
+		(property "Value" "MX-compatible"
 			(at 0 8 0)
 			(layer "F.Fab")
@@
 			)
 		)
-		(property "Value" "Redragon Low Profile switches"
+		(property "Value" "MX-compatible"
 			(at 0 8 0)
 			(layer "F.Fab")
@@
 			)
 		)
-		(property "Value" "Redragon Low Profile switches"
+		(property "Value" "MX-compatible"
 			(at 0 8 0)
 			(layer "F.Fab")
@@
 			)
 		)
-		(property "Value" "Redragon Low Profile switches"
+		(property "Value" "MX-compatible"
 			(at 0 8 0)
 			(layer "F.Fab")
@@
 			)
 		)
-		(property "Value" "Redragon Low Profile switches"
+		(property "Value" "MX-compatible"
 			(at 0 8 0)
 			(layer "F.Fab")
@@
 			)
 		)
-		(property "Value" "Redragon Low Profile switches"
+		(property "Value" "MX-compatible"
 			(at 0 8 0)
 			(layer "F.Fab")
@@
 			)
 		)
-		(property "Value" "Redragon Low Profile switches"
+		(property "Value" "MX-compatible"
 			(at 0 8 0)
 			(layer "F.Fab")
@@
 			)
 		)
-		(property "Value" "Redragon Low Profile switches"
+		(property "Value" "MX-compatible"
 			(at 0 8 0)
 			(layer "F.Fab")
@@
 			)
 		)
-		(property "Value" "Redragon Low Profile switches"
+		(property "Value" "MX-compatible"
 			(at 0 8 0)
 			(layer "F.Fab")
@@
 			)
 		)
-		(property "Value" "Redragon Low Profile switches"
+		(property "Value" "MX-compatible"
 			(at 0 8 0)
 			(layer "F.Fab")
@@
 			)
 		)
-		(property "Value" "Redragon Low Profile switches"
+		(property "Value" "MX-compatible"
 			(at 0 8 0)
 			(layer "F.Fab")
@@
 			)
 		)
-		(property "Value" "Redragon Low Profile switches"
+		(property "Value" "MX-compatible"
 			(at 0 8 0)
 			(layer "F.Fab")
@@
 			)
 		)
-		(property "Value" "Redragon Low Profile switches"
+		(property "Value" "MX-compatible"
 			(at 0 8 0)
 			(layer "F.Fab")
@@
 			)
 		)
-		(property "Value" "Redragon Low Profile switches"
+		(property "Value" "MX-compatible"
 			(at 0 8 0)
 			(layer "F.Fab")
@@
 			)
 		)
-		(property "Value" "Redragon Low Profile switches"
+		(property "Value" "MX-compatible"
 			(at 0 8 0)
 			(layer "F.Fab")

Commit message: pcb: tidy values in ch32x-48
Parts:
- C1, C2: value 100n -> 100nF
- J1: value USB_C_Receptacle_USB2.0 -> USB Type-C Female 16P
- R1, R4, R5: value 10K -> 10k
