File: pcb/keyboard-ch32x-48.kicad_sch (KiCad schematic)
At the start: 117 parts, among them J1 USB_C_Receptacle_USB2.0, J2 Conn_01x02, J3 Conn_01x04, SW1 SW_SPST, SW2 SW_SPST, U1 CH32X033F8P6

Commit message: pcb: ch32x-48 rev 2025.2
Parts:
- removed D_5_1, D_5_2, D_5_3, D_5_4, D_5_5, D_5_6, D_5_7, D_6_1, D_6_2, D_6_3, D_6_4, D_6_5, D_6_6, D_6_7, D_7_1, D_7_2, D_7_3, D_7_4, D_7_5, D_7_6: 1N4148, Diode_SMD:D_1206_3216Metric, symbol Device:D
- removed SW_5_1, SW_5_2, SW_5_3, SW_5_4, SW_5_5, SW_5_6, SW_5_7, SW_6_1, SW_6_2, SW_6_3, SW_6_4, SW_6_5, SW_6_6, SW_6_7, SW_7_1, SW_7_2, SW_7_3, SW_7_4, SW_7_5, SW_7_6: MX-compatible, ProjectLocal:SW_Cherry_MX_PCB_1.00u_BSilkRef, symbol Switch:SW_Push
- removed U1: CH32X033F8P6, Package_SO:TSSOP-20_4.4x6.5mm_P0.65mm, symbol ProjectLocal:CH32X033F8P6
- added D_1_10, D_1_11, D_1_12, D_1_8, D_1_9, D_2_10, D_2_11, D_2_12, D_2_8, D_2_9, D_3_10, D_3_11, D_3_12, D_3_8, D_3_9, D_4_10, D_4_11, D_4_12, D_4_8, D_4_9: 1N4148, Diode_SMD:D_1206_3216Metric, symbol Device:D
- added SW_1_10, SW_1_11, SW_1_12, SW_1_8, SW_1_9, SW_2_10, SW_2_11, SW_2_12, SW_2_8, SW_2_9, SW_3_10, SW_3_11, SW_3_12, SW_3_8, SW_3_9, SW_4_10, SW_4_11, SW_4_12, SW_4_8, SW_4_9: Redragon Low Profile switches, Switch_Keyboard_Cherry_MX:SW_Cherry_MX_PCB_1.00u, symbol Switch:SW_Push
- added U1: CH32X035C8T6, Package_QFP:LQFP-48_7x7mm_P0.5mm, symbol ProjectLocal:CH32X035C8T6
- SW_1_1, SW_1_2, SW_1_3, SW_1_4, SW_1_5, SW_1_6, SW_1_7, SW_2_1, SW_2_2, SW_2_3, SW_2_4, SW_2_5, SW_2_6, SW_2_7, SW_3_1, SW_3_2, SW_3_3, SW_3_4, SW_3_5, SW_3_6, SW_3_7, SW_4_1, SW_4_2, SW_4_3, SW_4_4, SW_4_5, SW_4_6, SW_4_7: value MX-compatible -> Redragon Low Profile switches; footprint ProjectLocal:SW_Cherry_MX_PCB_1.00u_BSilkRef -> Switch_Keyboard_Cherry_MX:SW_Cherry_MX_PCB_1.00u
Connections:
- net COL1: now also U1.31 (PB11)
- net COL2: now also U1.30 (PB10)
- net COL3: now also U1.29 (PB9)
- net COL4: now also U1.28 (PB8)
- net COL5: now also U1.27 (PB7)
- net COL6: now also U1.26 (PB6)
- net COL7: now also U1.9 (PA23)
- net DCK: now also U1.37 (PC19); no longer D_2_1.2 (A), D_2_2.2 (A), D_2_3.2 (A), D_2_4.2 (A), D_2_5.2 (A), D_2_6.2 (A), D_2_7.2 (A)
- net DIO: now also U1.34 (PC18)
- net DM: now also U1.32 (PC16)
- net DOWNLOAD: now also U1.33 (PC17)
- net GND: now also U1.47 (GND)
- net LED: now also U1.35 (PB12)
- net RESET: now also U1.7 (PA21)
- net ROW1: now also D_1_1.1 (K), D_1_2.1 (K), D_1_3.1 (K), D_1_4.1 (K), D_1_5.1 (K), D_1_6.1 (K), D_1_7.1 (K), D_1_10.1 (K), D_1_11.1 (K), D_1_12.1 (K), D_1_8.1 (K), D_1_9.1 (K), U1.40 (PA8); no longer D_1_1.2 (A), D_1_2.2 (A), D_1_3.2 (A), D_1_4.2 (A), D_1_5.2 (A), D_1_6.2 (A), D_1_7.2 (A)
- net ROW3: now also D_3_1.1 (K), D_3_2.1 (K), D_3_3.1 (K), D_3_4.1 (K), D_3_5.1 (K), D_3_6.1 (K), D_3_7.1 (K), D_3_10.1 (K), D_3_11.1 (K), D_3_12.1 (K), D_3_8.1 (K), D_3_9.1 (K), U1.14 (PA4); no longer D_3_1.2 (A), D_3_2.2 (A), D_3_3.2 (A), D_3_4.2 (A), D_3_5.2 (A), D_3_6.2 (A), D_3_7.2 (A), J2.2 (Pin_2)
- net ROW4: now also D_4_1.1 (K), D_4_2.1 (K), D_4_3.1 (K), D_4_4.1 (K), D_4_5.1 (K), D_4_6.1 (K), D_4_7.1 (K), D_4_10.1 (K), D_4_11.1 (K), D_4_12.1 (K), D_4_8.1 (K), D_4_9.1 (K), U1.16 (PA6); no longer D_4_1.2 (A), D_4_2.2 (A), D_4_3.2 (A), D_4_4.2 (A), D_4_5.2 (A), D_4_6.2 (A), D_4_7.2 (A), J2.1 (Pin_1)
- net VDD: now also U1.48 (VDD)
- net at SW_4_1.2: now also D_4_1.2 (A); no longer D_4_1.1 (K)
- net at SW_3_2.2: now also D_3_2.2 (A); no longer D_3_2.1 (K)
- net at SW_4_5.2: now also D_4_5.2 (A); no longer D_4_5.1 (K)
- net at SW_1_5.2: now also D_1_5.2 (A); no longer D_1_5.1 (K)
- net at SW_4_3.2: now also D_4_3.2 (A); no longer D_4_3.1 (K)
- net at SW_4_4.2: now also D_4_4.2 (A); no longer D_4_4.1 (K)
- net at SW_1_2.2: now also D_1_2.2 (A); no longer D_1_2.1 (K)
- net at SW_1_4.2: now also D_1_4.2 (A); no longer D_1_4.1 (K)
- net at SW_3_6.2: now also D_3_6.2 (A); no longer D_3_6.1 (K)
- net at SW_1_6.2: now also D_1_6.2 (A); no longer D_1_6.1 (K)
- net at SW_3_5.2: now also D_3_5.2 (A); no longer D_3_5.1 (K)
- net at SW_3_7.2: now also D_3_7.2 (A); no longer D_3_7.1 (K)
- net at SW_2_1.2: now also D_2_1.2 (A); no longer D_2_1.1 (K)
- net at SW_2_2.2: now also D_2_2.2 (A); no longer D_2_2.1 (K)
- net at SW_1_3.2: now also D_1_3.2 (A); no longer D_1_3.1 (K)
- net at SW_4_7.2: now also D_4_7.2 (A); no longer D_4_7.1 (K)
- net at SW_4_2.2: now also D_4_2.2 (A); no longer D_4_2.1 (K)
- net at SW_2_3.2: now also D_2_3.2 (A); no longer D_2_3.1 (K)
- net at SW_2_4.2: now also D_2_4.2 (A); no longer D_2_4.1 (K)
- net at SW_4_6.2: now also D_4_6.2 (A); no longer D_4_6.1 (K)
- net at SW_2_5.2: now also D_2_5.2 (A); no longer D_2_5.1 (K)
- net at SW_2_6.2: now also D_2_6.2 (A); no longer D_2_6.1 (K)
- net at SW_2_7.2: now also D_2_7.2 (A); no longer D_2_7.1 (K)
- net at SW_3_3.2: now also D_3_3.2 (A); no longer D_3_3.1 (K)
- net at SW_1_7.2: now also D_1_7.2 (A); no longer D_1_7.1 (K)
- net at SW_3_1.2: now also D_3_1.2 (A); no longer D_3_1.1 (K)
- net at SW_3_4.2: now also D_3_4.2 (A); no longer D_3_4.1 (K)
- net at SW_1_1.2: now also D_1_1.2 (A); no longer D_1_1.1 (K)
- new net: D_2_8.2 (A), SW_2_8.2
- new net: D_2_9.2 (A), SW_2_9.2
- new net: D_3_9.2 (A), SW_3_9.2
- new net: D_2_10.2 (A), SW_2_10.2
- new net: D_1_8.2 (A), SW_1_8.2
- new net: D_4_11.2 (A), SW_4_11.2
- new net: D_2_11.2 (A), SW_2_11.2
- new net: D_3_12.2 (A), SW_3_12.2
- new net: D_1_9.2 (A), SW_1_9.2
- new net: D_4_8.2 (A), SW_4_8.2
- new net: D_4_12.2 (A), SW_4_12.2
- new net: D_3_8.2 (A), SW_3_8.2
- new net: D_2_12.2 (A), SW_2_12.2
- new net: D_4_9.2 (A), SW_4_9.2
- new net: D_1_10.2 (A), SW_1_10.2
- new net: D_3_10.2 (A), SW_3_10.2
- new net: D_1_11.2 (A), SW_1_11.2
- new net: D_4_10.2 (A), SW_4_10.2
- new net: D_1_12.2 (A), SW_1_12.2
- new net: D_3_11.2 (A), SW_3_11.2
- new net COL10: SW_1_10.1, SW_2_10.1, SW_3_10.1, SW_4_10.1, U1.5 (PA19)
- new net COL11: SW_1_11.1, SW_2_11.1, SW_3_11.1, SW_4_11.1, U1.4 (PA18)
- new net COL12: SW_1_12.1, SW_2_12.1, SW_3_12.1, SW_4_12.1, U1.3 (PA17)
- new net COL8: SW_1_8.1, SW_2_8.1, SW_3_8.1, SW_4_8.1, U1.8 (PA22)
- new net COL9: SW_1_9.1, SW_2_9.1, SW_3_9.1, SW_4_9.1, U1.6 (PA20)
- new net ROW2: D_2_1.1 (K), D_2_10.1 (K), D_2_11.1 (K), D_2_12.1 (K), D_2_2.1 (K), D_2_3.1 (K), D_2_4.1 (K), D_2_5.1 (K), D_2_6.1 (K), D_2_7.1 (K), D_2_8.1 (K), D_2_9.1 (K), U1.12 (PA2)
- new net RX: J2.2 (Pin_2), U1.2 (PA16)
- new net TX: J2.1 (Pin_1), U1.1 (PA15)
- no-connect marks 2 -> 24
Other:
- note added: "- Constraints on pin output: None of PA7, PB0 used by matrix. (No constraint). - Constraints on pull-down input: All matrix rows are PA0-PA15. Can be used with pull-down input. Hence, the diodes in the matrix can be "col to row"."
- note added: "Switch Matrix The keyboard has 75 keys laid out in a 5-row-15-column grid."
- note removed: "- Constraints on pin output: Since PA7 is used as ROWx, matrix scanning MUST use rows as inputs. - Constraints on pull-down input: Since PC18,PC19 are used as ROWx, matrix scanning MUST pull up rows. Hence, the diodes in the matrix must be "row to col"."
- note removed: "NOTE: SWD (SDI) is enabled by default. This causes issues with matrix scanning on Row6. Refer to Reference Manual section on AFIO remap register for disabling SWD."
- note removed: "Switch Matrix The keyboard has 48 keys laid out in a 4-row-12-column grid. It uses fewer GPIO pins to have a 7x7 matrix (14 pins) than to use a 4x12 (16 pins) matrix. The mapping is top-to-bottom, left-to-right. This retains "column X <= Y". To find the key number: switch number = keyboard column * number of rows + keyboard row. To find the logical column, 'row': (switch number / 7, switch number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"
- moved on the sheet: SW_1_1, SW_2_1, SW_3_1, SW_4_1
