File: pcb/keyboard-ch32x-48.kicad_sch (KiCad schematic)
At the start: 117 parts, among them J1 USB_C_Receptacle_USB2.0, J2 Conn_01x02, J3 Conn_01x04, SW1 SW_SPST, SW2 SW_SPST, U1 CH32X035C8T6

Commit message: pcb: CH32X-48: fix incorrect value for SW_r_c
Parts:
- SW_1_1, SW_1_10, SW_1_11, SW_1_12, SW_1_2, SW_1_3, SW_1_4, SW_1_5, SW_1_6, SW_1_7, SW_1_8, SW_1_9, SW_2_1, SW_2_10, SW_2_11, SW_2_12, SW_2_2, SW_2_3, SW_2_4, SW_2_5, SW_2_6, SW_2_7, SW_2_8, SW_2_9, SW_3_1, SW_3_10, SW_3_11, SW_3_12, SW_3_2, SW_3_3, SW_3_4, SW_3_5, SW_3_6, SW_3_7, SW_3_8, SW_3_9, SW_4_1, SW_4_10, SW_4_11, SW_4_12, SW_4_2, SW_4_3, SW_4_4, SW_4_5, SW_4_6, SW_4_7, SW_4_8, SW_4_9: value Redragon Low Profile switches -> MX-compatible
Changed lines of the file:
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@@
 			)
 		)
-		(property "Value" "Redragon Low Profile switches"
+		(property "Value" "MX-compatible"
 			(at 154.94 97.9424 0)
 			(hide yes)
@@
 			)
 		)
-		(property "Value" "Redragon Low Profile switches"
+		(property "Value" "MX-compatible"
 			(at 200.66 97.9424 0)
 			(hide yes)
@@
 			)
 		)
-		(property "Value" "Redragon Low Profile switches"
+		(property "Value" "MX-compatible"
 			(at 139.7 114.4524 0)
 			(hide yes)
@@
 			)
 		)
-		(property "Value" "Redragon Low Profile switches"
+		(property "Value" "MX-compatible"
 			(at 185.42 130.9624 0)
 			(hide yes)
@@
 			)
 		)
-		(property "Value" "Redragon Low Profile switches"
+		(property "Value" "MX-compatible"
 			(at 261.62 130.9624 0)
 			(hide yes)
@@
 			)
 		)
-		(property "Value" "Redragon Low Profile switches"
+		(property "Value" "MX-compatible"
 			(at 246.38 97.9424 0)
 			(hide yes)
@@
 			)
 		)
-		(property "Value" "Redragon Low Profile switches"
+		(property "Value" "MX-compatible"
 			(at 215.9 97.9424 0)
 			(hide yes)
@@
 			)
 		)
-		(property "Value" "Redragon Low Profile switches"
+		(property "Value" "MX-compatible"
 			(at 124.46 114.4524 0)
 			(hide yes)
@@
 			)
 		)
-		(property "Value" "Redragon Low Profile switches"
+		(property "Value" "MX-compatible"
 			(at 261.62 97.9424 0)
 			(hide yes)
@@
 			)
 		)
-		(property "Value" "Redragon Low Profile switches"
+		(property "Value" "MX-compatible"
 			(at 276.86 114.4524 0)
 			(hide yes)
@@
 			)
 		)
-		(property "Value" "Redragon Low Profile switches"
+		(property "Value" "MX-compatible"
 			(at 124.46 97.9424 0)
 			(hide yes)
@@
 			)
 		)
-		(property "Value" "Redragon Low Profile switches"
+		(property "Value" "MX-compatible"
 			(at 185.42 114.4524 0)
 			(hide yes)
@@
 			)
 		)
-		(property "Value" "Redragon Low Profile switches"
+		(property "Value" "MX-compatible"
 			(at 124.46 81.4324 0)
 			(hide yes)
@@
 			)
 		)
-		(property "Value" "Redragon Low Profile switches"
+		(property "Value" "MX-compatible"
 			(at 215.9 130.9624 0)
 			(hide yes)
@@
 			)
 		)
-		(property "Value" "Redragon Low Profile switches"
+		(property "Value" "MX-compatible"
 			(at 276.86 97.9424 0)
 			(hide yes)
@@
 			)
 		)
-		(property "Value" "Redragon Low Profile switches"
+		(property "Value" "MX-compatible"
 			(at 109.22 97.9424 0)
 			(hide yes)
@@
 			)
 		)
-		(property "Value" "Redragon Low Profile switches"
+		(property "Value" "MX-compatible"
 			(at 246.38 114.4524 0)
 			(hide yes)
@@
 			)
 		)
-		(property "Value" "Redragon Low Profile switches"
+		(property "Value" "MX-compatible"
 			(at 261.62 81.4324 0)
 			(hide yes)
@@
 			)
 		)
-		(property "Value" "Redragon Low Profile switches"
+		(property "Value" "MX-compatible"
 			(at 200.66 81.4324 0)
 			(hide yes)
@@
 			)
 		)
-		(property "Value" "Redragon Low Profile switches"
+		(property "Value" "MX-compatible"
 			(at 200.66 114.4524 0)
 			(hide yes)
@@
 			)
 		)
-		(property "Value" "Redragon Low Profile switches"
+		(property "Value" "MX-compatible"
 			(at 139.7 81.4324 0)
 			(hide yes)
@@
 			)
 		)
-		(property "Value" "Redragon Low Profile switches"
+		(property "Value" "MX-compatible"
 			(at 139.7 97.9424 0)
 			(hide yes)
@@
 			)
 		)
-		(property "Value" "Redragon Low Profile switches"
+		(property "Value" "MX-compatible"
 			(at 231.14 114.4524 0)
 			(hide yes)
@@
 			)
 		)
-		(property "Value" "Redragon Low Profile switches"
+		(property "Value" "MX-compatible"
 			(at 276.86 130.9624 0)
 			(hide yes)
@@
 			)
 		)
-		(property "Value" "Redragon Low Profile switches"
+		(property "Value" "MX-compatible"
 			(at 276.86 81.4324 0)
 			(hide yes)
@@
 			)
 		)
-		(property "Value" "Redragon Low Profile switches"
+		(property "Value" "MX-compatible"
 			(at 231.14 130.9624 0)
 			(hide yes)
@@
 			)
 		)
-		(property "Value" "Redragon Low Profile switches"
+		(property "Value" "MX-compatible"
 			(at 185.42 81.4324 0)
 			(hide yes)
@@
 			)
 		)
-		(property "Value" "Redragon Low Profile switches"
+		(property "Value" "MX-compatible"
 			(at 124.46 130.9624 0)
 			(hide yes)
@@
 			)
 		)
-		(property "Value" "Redragon Low Profile switches"
+		(property "Value" "MX-compatible"
 			(at 154.94 114.4524 0)
 			(hide yes)
@@
 			)
 		)
-		(property "Value" "Redragon Low Profile switches"
+		(property "Value" "MX-compatible"
 			(at 261.62 114.4524 0)
 			(hide yes)
@@
 			)
 		)
-		(property "Value" "Redragon Low Profile switches"
+		(property "Value" "MX-compatible"
 			(at 246.38 130.9624 0)
 			(hide yes)
@@
 			)
 		)
-		(property "Value" "Redragon Low Profile switches"
+		(property "Value" "MX-compatible"
 			(at 170.18 81.4324 0)
 			(hide yes)
@@
 			)
 		)
-		(property "Value" "Redragon Low Profile switches"
+		(property "Value" "MX-compatible"
 			(at 200.66 130.9624 0)
 			(hide yes)
@@
 			)
 		)
-		(property "Value" "Redragon Low Profile switches"
+		(property "Value" "MX-compatible"
 			(at 109.22 114.4524 0)
 			(hide yes)
@@
 			)
 		)
-		(property "Value" "Redragon Low Profile switches"
+		(property "Value" "MX-compatible"
 			(at 231.14 81.4324 0)
 			(hide yes)
@@
 			)
 		)
-		(property "Value" "Redragon Low Profile switches"
+		(property "Value" "MX-compatible"
 			(at 170.18 130.9624 0)
 			(hide yes)
@@
 			)
 		)
-		(property "Value" "Redragon Low Profile switches"
+		(property "Value" "MX-compatible"
 			(at 215.9 114.4524 0)
 			(hide yes)
@@
 			)
 		)
-		(property "Value" "Redragon Low Profile switches"
+		(property "Value" "MX-compatible"
 			(at 154.94 81.4324 0)
 			(hide yes)
@@
 			)
 		)
-		(property "Value" "Redragon Low Profile switches"
+		(property "Value" "MX-compatible"
 			(at 231.14 97.9424 0)
 			(hide yes)
@@
 			)
 		)
-		(property "Value" "Redragon Low Profile switches"
+		(property "Value" "MX-compatible"
 			(at 109.22 81.4324 0)
 			(hide yes)
@@
 			)
 		)
-		(property "Value" "Redragon Low Profile switches"
+		(property "Value" "MX-compatible"
 			(at 185.42 97.9424 0)
 			(hide yes)
@@
 			)
 		)
-		(property "Value" "Redragon Low Profile switches"
+		(property "Value" "MX-compatible"
 			(at 139.7 130.9624 0)
 			(hide yes)
@@
 			)
 		)
-		(property "Value" "Redragon Low Profile switches"
+		(property "Value" "MX-compatible"
 			(at 109.22 130.9624 0)
 			(hide yes)
@@
 			)
 		)
-		(property "Value" "Redragon Low Profile switches"
+		(property "Value" "MX-compatible"
 			(at 215.9 81.4324 0)
 			(hide yes)
@@
 			)
 		)
-		(property "Value" "Redragon Low Profile switches"
+		(property "Value" "MX-compatible"
 			(at 170.18 114.4524 0)
 			(hide yes)
@@
 			)
 		)
-		(property "Value" "Redragon Low Profile switches"
+		(property "Value" "MX-compatible"
 			(at 170.18 97.9424 0)
 			(hide yes)
@@
 			)
 		)
-		(property "Value" "Redragon Low Profile switches"
+		(property "Value" "MX-compatible"
 			(at 154.94 130.9624 0)
 			(hide yes)
@@
 			)
 		)
-		(property "Value" "Redragon Low Profile switches"
+		(property "Value" "MX-compatible"
 			(at 246.38 81.4324 0)
 			(hide yes)

Commit message: pcb: tidy values in ch32x-48
Parts:
- C1, C2: value 100n -> 100nF; LCSC C49678 -> (none)
- C3: LCSC C49678 -> (none)
- D_1_1, D_1_10, D_1_11, D_1_12, D_1_2, D_1_3, D_1_4, D_1_5, D_1_6, D_1_7, D_1_8, D_1_9, D_2_1, D_2_10, D_2_11, D_2_12, D_2_2, D_2_3, D_2_4, D_2_5, D_2_6, D_2_7, D_2_8, D_2_9, D_3_1, D_3_10, D_3_11, D_3_12, D_3_2, D_3_3, D_3_4, D_3_5, D_3_6, D_3_7, D_3_8, D_3_9, D_4_1, D_4_10, D_4_11, D_4_12, D_4_2, D_4_3, D_4_4, D_4_5, D_4_6, D_4_7, D_4_8, D_4_9: LCSC C9808 -> (none)
- J1: value USB_C_Receptacle_USB2.0 -> USB Type-C Female 16P
- R1, R4, R5: value 10K -> 10k; LCSC C17414 -> (none)
- R2, R3: LCSC C27834 -> (none)
Changed lines of the file:
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@@
 			)
 		)
-		(property "LCSC" "C9808"
+		(property "LCSC" ""
 			(at 144.78 90.17 0)
 			(hide yes)
@@
 			)
 		)
-		(property "LCSC" "C9808"
+		(property "LCSC" ""
 			(at 114.3 139.7 0)
 			(hide yes)
@@
 			)
 		)
-		(property "Value" "10K"
+		(property "Value" "10k"
 			(at 201.93 158.75 90)
 			(show_name no)
@@
 			)
 		)
-		(property "LCSC" "C17414"
+		(property "LCSC" ""
 			(at 201.93 162.56 0)
 			(hide yes)
@@
 			)
 		)
-		(property "LCSC" "C9808"
+		(property "LCSC" ""
 			(at 220.98 106.68 0)
 			(hide yes)
@@
 			)
 		)
-		(property "LCSC" "C9808"
+		(property "LCSC" ""
 			(at 160.02 123.19 0)
 			(hide yes)
@@
 			)
 		)
-		(property "LCSC" "C9808"
+		(property "LCSC" ""
 			(at 236.22 106.68 0)
 			(hide yes)
@@
 			)
 		)
-		(property "LCSC" "C9808"
+		(property "LCSC" ""
 			(at 236.22 123.19 0)
 			(hide yes)
@@
 			)
 		)
-		(property "LCSC" "C9808"
+		(property "LCSC" ""
 			(at 251.46 106.68 0)
 			(hide yes)
@@
 			)
 		)
-		(property "LCSC" "C9808"
+		(property "LCSC" ""
 			(at 220.98 90.17 0)
 			(hide yes)
@@
 			)
 		)
-		(property "LCSC" "C9808"
+		(property "LCSC" ""
 			(at 205.74 106.68 0)
 			(hide yes)
@@
 			)
 		)
-		(property "LCSC" "C27834"
+		(property "LCSC" ""
 			(at 54.61 109.22 0)
 			(hide yes)
@@
 			)
 		)
-		(property "LCSC" "C9808"
+		(property "LCSC" ""
 			(at 129.54 139.7 0)
 			(hide yes)
@@
 			)
 		)
-		(property "LCSC" "C9808"
+		(property "LCSC" ""
 			(at 236.22 90.17 0)
 			(hide yes)
@@
 			)
 		)
-		(property "LCSC" "C9808"
+		(property "LCSC" ""
 			(at 144.78 106.68 0)
 			(hide yes)
@@
 			)
 		)
-		(property "Value" "100n"
+		(property "Value" "100nF"
 			(at 50.8 163.83 0)
 			(show_name no)
@@
 			)
 		)
-		(property "LCSC" "C49678"
+		(property "LCSC" ""
 			(at 46.99 162.56 0)
 			(hide yes)
@@
 			)
 		)
-		(property "LCSC" "C9808"
+		(property "LCSC" ""
 			(at 281.94 139.7 0)
 			(hide yes)
@@
 			)
 		)
-		(property "LCSC" "C9808"
+		(property "LCSC" ""
 			(at 220.98 123.19 0)
 			(hide yes)
@@
 			)
 		)
-		(property "Value" "USB_C_Receptacle_USB2.0"
+		(property "Value" "USB Type-C Female 16P"
 			(at 30.48 92.71 0)
 			(show_name no)
@@
 			)
 		)
-		(property "LCSC" "C9808"
+		(property "LCSC" ""
 			(at 220.98 139.7 0)
 			(hide yes)
@@
 			)
 		)
-		(property "LCSC" "C9808"
+		(property "LCSC" ""
 			(at 205.74 90.17 0)
 			(hide yes)
@@
 			)
 		)
-		(property "Value" "100n"
+		(property "Value" "100nF"
 			(at 48.26 74.93 0)
 			(show_name no)
@@
 			)
 		)
-		(property "LCSC" "C49678"
+		(property "LCSC" ""
 			(at 44.45 73.66 0)
 			(hide yes)
@@
 			)
 		)
-		(property "LCSC" "C9808"
+		(property "LCSC" ""
 			(at 144.78 139.7 0)
 			(hide yes)
@@
 			)
 		)
-		(property "LCSC" "C9808"
+		(property "LCSC" ""
 			(at 129.54 90.17 0)
 			(hide yes)
@@
 			)
 		)
-		(property "LCSC" "C9808"
+		(property "LCSC" ""
 			(at 114.3 106.68 0)
 			(hide yes)
@@
 			)
 		)
-		(property "LCSC" "C9808"
+		(property "LCSC" ""
 			(at 236.22 139.7 0)
 			(hide yes)
@@
 			)
 		)
-		(property "LCSC" "C9808"
+		(property "LCSC" ""
 			(at 251.46 90.17 0)
 			(hide yes)
@@
 			)
 		)
-		(property "LCSC" "C9808"
+		(property "LCSC" ""
 			(at 205.74 123.19 0)
 			(hide yes)
@@
 			)
 		)
-		(property "LCSC" "C9808"
+		(property "LCSC" ""
 			(at 144.78 123.19 0)
 			(hide yes)
@@
 			)
 		)
-		(property "LCSC" "C9808"
+		(property "LCSC" ""
 			(at 251.46 123.19 0)
 			(hide yes)
@@
 			)
 		)
-		(property "LCSC" "C9808"
+		(property "LCSC" ""
 			(at 205.74 139.7 0)
 			(hide yes)
@@
 			)
 		)
-		(property "LCSC" "C49678"
+		(property "LCSC" ""
 			(at 58.42 73.66 0)
 			(hide yes)
@@
 			)
 		)
-		(property "Value" "10K"
+		(property "Value" "10k"
 			(at 58.42 187.96 90)
 			(show_name no)
@@
 			)
 		)
-		(property "LCSC" "C17414"
+		(property "LCSC" ""
 			(at 58.42 191.77 0)
 			(hide yes)
@@
 			)
 		)
-		(property "LCSC" "C9808"
+		(property "LCSC" ""
 			(at 190.5 106.68 0)
 			(hide yes)
@@
 			)
 		)
-		(property "LCSC" "C9808"
+		(property "LCSC" ""
 			(at 251.46 139.7 0)
 			(hide yes)
@@
 			)
 		)
-		(property "LCSC" "C9808"
+		(property "LCSC" ""
 			(at 160.02 106.68 0)
 			(hide yes)
@@
 			)
 		)
-		(property "LCSC" "C9808"
+		(property "LCSC" ""
 			(at 190.5 90.17 0)
 			(hide yes)
@@
 			)
 		)
-		(property "LCSC" "C9808"
+		(property "LCSC" ""
 			(at 129.54 106.68 0)
 			(hide yes)
@@
 			)
 		)
-		(property "LCSC" "C9808"
+		(property "LCSC" ""
 			(at 190.5 139.7 0)
 			(hide yes)
@@
 			)
 		)
-		(property "LCSC" "C9808"
+		(property "LCSC" ""
 			(at 266.7 123.19 0)
 			(hide yes)
@@
 			)
 		)
-		(property "Value" "10K"
+		(property "Value" "10k"
 			(at 232.41 158.75 90)
 			(show_name no)
@@
 			)
 		)
-		(property "LCSC" "C17414"
+		(property "LCSC" ""
 			(at 232.41 162.56 0)
 			(hide yes)
@@
 			)
 		)
-		(property "LCSC" "C9808"
+		(property "LCSC" ""
 			(at 114.3 123.19 0)
 			(hide yes)
@@
 			)
 		)
-		(property "LCSC" "C9808"
+		(property "LCSC" ""
 			(at 160.02 139.7 0)
 			(hide yes)
@@
 			)
 		)
-		(property "LCSC" "C9808"
+		(property "LCSC" ""
 			(at 175.26 123.19 0)
 			(hide yes)
@@
 			)
 		)
-		(property "LCSC" "C27834"
+		(property "LCSC" ""
 			(at 64.77 109.22 0)
 			(hide yes)
@@
 			)
 		)
-		(property "LCSC" "C9808"
+		(property "LCSC" ""
 			(at 129.54 123.19 0)
 			(hide yes)
@@
 			)
 		)
-		(property "LCSC" "C9808"
+		(property "LCSC" ""
 			(at 160.02 90.17 0)
 			(hide yes)
@@
 			)
 		)
-		(property "LCSC" "C9808"
+		(property "LCSC" ""
 			(at 175.26 106.68 0)
 			(hide yes)
@@
 			)
 		)
-		(property "LCSC" "C9808"
+		(property "LCSC" ""
 			(at 281.94 106.68 0)
 			(hide yes)
@@
 			)
 		)
-		(property "LCSC" "C9808"
+		(property "LCSC" ""
 			(at 281.94 90.17 0)
 			(hide yes)
@@
 			)
 		)
-		(property "LCSC" "C9808"
+		(property "LCSC" ""
 			(at 266.7 90.17 0)
 			(hide yes)
@@
 			)
 		)
-		(property "LCSC" "C9808"
+		(property "LCSC" ""
 			(at 266.7 139.7 0)
 			(hide yes)
@@
 			)
 		)
-		(property "LCSC" "C9808"
+		(property "LCSC" ""
 			(at 175.26 90.17 0)
 			(hide yes)
@@
 			)
 		)
-		(property "LCSC" "C9808"
+		(property "LCSC" ""
 			(at 281.94 123.19 0)
 			(hide yes)
@@
 			)
 		)
-		(property "LCSC" "C9808"
+		(property "LCSC" ""
 			(at 190.5 123.19 0)
 			(hide yes)
@@
 			)
 		)
-		(property "LCSC" "C9808"
+		(property "LCSC" ""
 			(at 175.26 139.7 0)
 			(hide yes)
@@
 			)
 		)
-		(property "LCSC" "C9808"
+		(property "LCSC" ""
 			(at 114.3 90.17 0)
 			(hide yes)
@@
 			)
 		)
-		(property "LCSC" "C9808"
+		(property "LCSC" ""
 			(at 266.7 106.68 0)
 			(hide yes)

Commit message: pcb: tidy layout of CH32X-48 schematic
Other:
- note added: "Switch Matrix The keyboard has 48 keys laid out in a 4-row-12-column grid."
- note removed: "Switch Matrix The keyboard has 75 keys laid out in a 5-row-15-column grid."
- moved on the sheet: C2, C3, J1, R2, R3, U1

Commit message: pcb: update comment
Other:
- note added: "UART For simple printf debugging with UART2."
- note added: "WCH Link interface (CH32X033 only compatible with WCH-LinkE or WCH-LinkW)"
- note removed: "UART For simple printf debugging with UART2. ("ROW4"/SW_4_x switches can't be used while using UART2)."
- note removed: "WCH Link interface (CH32X033 only compatible with WCH-LinkE or WCH-LinkW) Using DIO/DCK prevents use of ROW2/ROW6. SWD (SDI) enabled by default; must be disabled after reset."
Changed lines of the file:
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@@
 		)
 	)
-	(text "WCH Link interface\n(CH32X033 only compatible with WCH-LinkE or WCH-LinkW)\nUsing DIO/DCK prevents use of ROW2/ROW6.\nSWD (SDI) enabled by default; must be disabled after reset."
+	(text "WCH Link interface\n(CH32X033 only compatible with WCH-LinkE or WCH-LinkW)"
 		(exclude_from_sim no)
 		(at 92.202 179.324 0)
@@
 		)
 	)
-	(text "UART\nFor simple printf debugging with UART2.\n(\"ROW4\"/SW_4_x switches can't be used\n while using UART2)."
+	(text "UART\nFor simple printf debugging with UART2."
 		(exclude_from_sim no)
 		(at 91.694 157.734 0)
