File: pcb/demo-usb-16pin.kicad_sch (KiCad schematic)
At the start: 7 parts, among them J1 USB_C_Receptacle_USB2.0, J2 Conn_01x04_Female, J3 Conn_01x04_Female, J4 Conn_01x10_Female

Commit message: pcb: tidy values in demo-usb-16pin
Parts:
- J1: value USB_C_Receptacle_USB2.0 -> USB Type-C Female 16P
- R1, R2: value 5.1K -> 5.1k
Changed lines of the file:
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@@
 			)
 		)
-		(property "Value" "USB_C_Receptacle_USB2.0"
+		(property "Value" "USB Type-C Female 16P"
 			(at 33.1978 28.5496 0)
 			(show_name no)
@@
 			)
 		)
-		(property "Value" "5.1K"
+		(property "Value" "5.1k"
 			(at 69.088 63.373 0)
 			(show_name no)
@@
 			)
 		)
-		(property "Value" "5.1K"
+		(property "Value" "5.1k"
 			(at 79.248 63.373 0)
 			(show_name no)
