File: pcb/keyboard-ch552-48.kicad_sch (KiCad schematic)
At the start: 113 parts, among them J1 USB_C_Receptacle_USB2.0, J2 Conn_01x06, SW1 SW_SPST, SW2 SW_SPST, U1 CH552T

Commit message: pcb: tidy values in ch552-48
Parts:
- C1, C2, C3: value 100n -> 100nF; LCSC C49678 -> (none)
- D_1_1, D_1_2, D_1_3, D_1_4, D_1_5, D_1_6, D_1_7, D_2_1, D_2_2, D_2_3, D_2_4, D_2_5, D_2_6, D_2_7, D_3_1, D_3_2, D_3_3, D_3_4, D_3_5, D_3_6, D_3_7, D_4_1, D_4_2, D_4_3, D_4_4, D_4_5, D_4_6, D_4_7, D_5_1, D_5_2, D_5_3, D_5_4, D_5_5, D_5_6, D_5_7, D_6_1, D_6_2, D_6_3, D_6_4, D_6_5, D_6_6, D_6_7, D_7_1, D_7_2, D_7_3, D_7_4, D_7_5, D_7_6: LCSC C9808 -> (none)
- J1: value USB_C_Receptacle_USB2.0 -> USB Type-C Female 16P
- R1: LCSC C17630 -> (none)
- R2: value 10K -> 10k; LCSC C17414 -> (none)
- R3, R4: LCSC C27834 -> (none)
Changed lines of the file:
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@@
 			)
 		)
-		(property "LCSC" "C9808"
+		(property "LCSC" ""
 			(at 187.96 85.09 0)
 			(hide yes)
@@
 			)
 		)
-		(property "LCSC" "C9808"
+		(property "LCSC" ""
 			(at 203.2 118.11 0)
 			(hide yes)
@@
 			)
 		)
-		(property "LCSC" "C9808"
+		(property "LCSC" ""
 			(at 248.92 85.09 0)
 			(hide yes)
@@
 			)
 		)
-		(property "LCSC" "C9808"
+		(property "LCSC" ""
 			(at 248.92 35.56 0)
 			(hide yes)
@@
 			)
 		)
-		(property "LCSC" "C9808"
+		(property "LCSC" ""
 			(at 218.44 85.09 0)
 			(hide yes)
@@
 			)
 		)
-		(property "LCSC" "C27834"
+		(property "LCSC" ""
 			(at 58.42 78.74 0)
 			(hide yes)
@@
 			)
 		)
-		(property "LCSC" "C9808"
+		(property "LCSC" ""
 			(at 187.96 134.62 0)
 			(hide yes)
@@
 			)
 		)
-		(property "LCSC" "C9808"
+		(property "LCSC" ""
 			(at 264.16 68.58 0)
 			(hide yes)
@@
 			)
 		)
-		(property "LCSC" "C9808"
+		(property "LCSC" ""
 			(at 248.92 134.62 0)
 			(hide yes)
@@
 			)
 		)
-		(property "LCSC" "C9808"
+		(property "LCSC" ""
 			(at 218.44 134.62 0)
 			(hide yes)
@@
 			)
 		)
-		(property "LCSC" "C9808"
+		(property "LCSC" ""
 			(at 233.68 85.09 0)
 			(hide yes)
@@
 			)
 		)
-		(property "LCSC" "C9808"
+		(property "LCSC" ""
 			(at 264.16 134.62 0)
 			(hide yes)
@@
 			)
 		)
-		(property "LCSC" "C9808"
+		(property "LCSC" ""
 			(at 233.68 101.6 0)
 			(hide yes)
@@
 			)
 		)
-		(property "LCSC" "C9808"
+		(property "LCSC" ""
 			(at 279.4 118.11 0)
 			(hide yes)
@@
 			)
 		)
-		(property "LCSC" "C9808"
+		(property "LCSC" ""
 			(at 248.92 68.58 0)
 			(hide yes)
@@
 			)
 		)
-		(property "Value" "100n"
+		(property "Value" "100nF"
 			(at 33.02 163.83 0)
 			(show_name no)
@@
 			)
 		)
-		(property "LCSC" "C49678"
+		(property "LCSC" ""
 			(at 29.21 162.56 0)
 			(hide yes)
@@
 			)
 		)
-		(property "LCSC" "C9808"
+		(property "LCSC" ""
 			(at 233.68 134.62 0)
 			(hide yes)
@@
 			)
 		)
-		(property "Value" "USB_C_Receptacle_USB2.0"
+		(property "Value" "USB Type-C Female 16P"
 			(at 34.29 62.23 0)
 			(show_name no)
@@
 			)
 		)
-		(property "LCSC" "C9808"
+		(property "LCSC" ""
 			(at 279.4 68.58 0)
 			(hide yes)
@@
 			)
 		)
-		(property "Value" "100n"
+		(property "Value" "100nF"
 			(at 33.02 129.54 0)
 			(show_name no)
@@
 			)
 		)
-		(property "LCSC" "C49678"
+		(property "LCSC" ""
 			(at 29.21 128.27 0)
 			(hide yes)
@@
 			)
 		)
-		(property "LCSC" "C9808"
+		(property "LCSC" ""
 			(at 264.16 118.11 0)
 			(hide yes)
@@
 			)
 		)
-		(property "LCSC" "C9808"
+		(property "LCSC" ""
 			(at 203.2 52.07 0)
 			(hide yes)
@@
 			)
 		)
-		(property "LCSC" "C17630"
+		(property "LCSC" ""
 			(at 43.18 158.75 0)
 			(hide yes)
@@
 			)
 		)
-		(property "LCSC" "C9808"
+		(property "LCSC" ""
 			(at 187.96 52.07 0)
 			(hide yes)
@@
 			)
 		)
-		(property "Value" "100n"
+		(property "Value" "100nF"
 			(at 45.72 129.54 0)
 			(show_name no)
@@
 			)
 		)
-		(property "LCSC" "C49678"
+		(property "LCSC" ""
 			(at 41.91 128.27 0)
 			(hide yes)
@@
 			)
 		)
-		(property "LCSC" "C9808"
+		(property "LCSC" ""
 			(at 248.92 118.11 0)
 			(hide yes)
@@
 			)
 		)
-		(property "LCSC" "C9808"
+		(property "LCSC" ""
 			(at 218.44 52.07 0)
 			(hide yes)
@@
 			)
 		)
-		(property "LCSC" "C9808"
+		(property "LCSC" ""
 			(at 203.2 134.62 0)
 			(hide yes)
@@
 			)
 		)
-		(property "LCSC" "C9808"
+		(property "LCSC" ""
 			(at 233.68 52.07 0)
 			(hide yes)
@@
 			)
 		)
-		(property "LCSC" "C9808"
+		(property "LCSC" ""
 			(at 203.2 101.6 0)
 			(hide yes)
@@
 			)
 		)
-		(property "LCSC" "C9808"
+		(property "LCSC" ""
 			(at 279.4 85.09 0)
 			(hide yes)
@@
 			)
 		)
-		(property "LCSC" "C9808"
+		(property "LCSC" ""
 			(at 248.92 101.6 0)
 			(hide yes)
@@
 			)
 		)
-		(property "LCSC" "C9808"
+		(property "LCSC" ""
 			(at 218.44 35.56 0)
 			(hide yes)
@@
 			)
 		)
-		(property "LCSC" "C9808"
+		(property "LCSC" ""
 			(at 203.2 68.58 0)
 			(hide yes)
@@
 			)
 		)
-		(property "LCSC" "C9808"
+		(property "LCSC" ""
 			(at 279.4 101.6 0)
 			(hide yes)
@@
 			)
 		)
-		(property "Value" "10K"
+		(property "Value" "10k"
 			(at 48.26 182.88 90)
 			(show_name no)
@@
 			)
 		)
-		(property "LCSC" "C17414"
+		(property "LCSC" ""
 			(at 48.26 186.69 0)
 			(hide yes)
@@
 			)
 		)
-		(property "LCSC" "C9808"
+		(property "LCSC" ""
 			(at 279.4 52.07 0)
 			(hide yes)
@@
 			)
 		)
-		(property "LCSC" "C9808"
+		(property "LCSC" ""
 			(at 233.68 35.56 0)
 			(hide yes)
@@
 			)
 		)
-		(property "LCSC" "C9808"
+		(property "LCSC" ""
 			(at 248.92 52.07 0)
 			(hide yes)
@@
 			)
 		)
-		(property "LCSC" "C9808"
+		(property "LCSC" ""
 			(at 187.96 101.6 0)
 			(hide yes)
@@
 			)
 		)
-		(property "LCSC" "C9808"
+		(property "LCSC" ""
 			(at 279.4 35.56 0)
 			(hide yes)
@@
 			)
 		)
-		(property "LCSC" "C9808"
+		(property "LCSC" ""
 			(at 187.96 118.11 0)
 			(hide yes)
@@
 			)
 		)
-		(property "LCSC" "C9808"
+		(property "LCSC" ""
 			(at 187.96 68.58 0)
 			(hide yes)
@@
 			)
 		)
-		(property "LCSC" "C9808"
+		(property "LCSC" ""
 			(at 233.68 68.58 0)
 			(hide yes)
@@
 			)
 		)
-		(property "LCSC" "C9808"
+		(property "LCSC" ""
 			(at 218.44 101.6 0)
 			(hide yes)
@@
 			)
 		)
-		(property "LCSC" "C9808"
+		(property "LCSC" ""
 			(at 203.2 85.09 0)
 			(hide yes)
@@
 			)
 		)
-		(property "LCSC" "C27834"
+		(property "LCSC" ""
 			(at 68.58 78.74 0)
 			(hide yes)
@@
 			)
 		)
-		(property "LCSC" "C9808"
+		(property "LCSC" ""
 			(at 264.16 101.6 0)
 			(hide yes)
@@
 			)
 		)
-		(property "LCSC" "C9808"
+		(property "LCSC" ""
 			(at 218.44 118.11 0)
 			(hide yes)
@@
 			)
 		)
-		(property "LCSC" "C9808"
+		(property "LCSC" ""
 			(at 264.16 35.56 0)
 			(hide yes)
@@
 			)
 		)
-		(property "LCSC" "C9808"
+		(property "LCSC" ""
 			(at 233.68 118.11 0)
 			(hide yes)
@@
 			)
 		)
-		(property "LCSC" "C9808"
+		(property "LCSC" ""
 			(at 203.2 35.56 0)
 			(hide yes)
@@
 			)
 		)
-		(property "LCSC" "C9808"
+		(property "LCSC" ""
 			(at 264.16 85.09 0)
 			(hide yes)
@@
 			)
 		)
-		(property "LCSC" "C9808"
+		(property "LCSC" ""
 			(at 264.16 52.07 0)
 			(hide yes)
@@
 			)
 		)
-		(property "LCSC" "C9808"
+		(property "LCSC" ""
 			(at 218.44 68.58 0)
 			(hide yes)
@@
 			)
 		)
-		(property "LCSC" "C9808"
+		(property "LCSC" ""
 			(at 187.96 35.56 0)
 			(hide yes)
