File: pcb/keyboard-ch552-36-rhs.kicad_pcb (KiCad board)
At the start: 2 copper layers, 100 x 96.5 mm, 55 parts, among them J1 USB Type-C Receptacle 12-pin, J2 PJ-320A, SW1 SW_SPST, SW2 SW_SPST, U1 CH552T

Commit message: pcb: tidy values in ch552-36
Parts:
- C1, C2, C3: value 100n -> 100nF
- R4: value 10K -> 10k
