File: pcb/keyboard-ch552-36-rhs.kicad_sch (KiCad schematic)
At the start: 56 parts, among them J1 PJ-320A, J1 USB Type-C Receptacle 12-pin, J3 Conn_01x06, SW1 SW_SPST, SW2 SW_SPST, U1 CH552T

Commit message: pcb: upgrade to kicad 10: keyboard-ch552-36
Parts:
- renumbered J1 to J2, R1 to R5, R2 to R6

Commit message: pcb: tidy values in ch552-36
Parts:
- C1, C2, C3: value 100n -> 100nF; LCSC C49678 -> (none)
- D_1_1, D_1_2, D_1_3, D_1_4, D_1_5, D_2_1, D_2_2, D_2_3, D_2_4, D_2_5, D_3_1, D_3_2, D_3_3, D_3_4, D_3_5, D_4_3, D_4_4, D_4_5: LCSC C9808 -> (none)
- R1, R2: LCSC C27834 -> (none)
- R3: LCSC C17630 -> (none)
- R4: value 10K -> 10k; LCSC C17414 -> (none)
Changed lines of the file:
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@@
 			)
 		)
-		(property "LCSC" "C9808"
+		(property "LCSC" ""
 			(at 248.92 85.09 0)
 			(hide yes)
@@
 			)
 		)
-		(property "LCSC" "C9808"
+		(property "LCSC" ""
 			(at 248.92 35.56 0)
 			(hide yes)
@@
 			)
 		)
-		(property "LCSC" "C9808"
+		(property "LCSC" ""
 			(at 218.44 85.09 0)
 			(hide yes)
@@
 			)
 		)
-		(property "LCSC" "C27834"
+		(property "LCSC" ""
 			(at 58.42 78.74 0)
 			(hide yes)
@@
 			)
 		)
-		(property "LCSC" "C9808"
+		(property "LCSC" ""
 			(at 233.68 85.09 0)
 			(hide yes)
@@
 			)
 		)
-		(property "LCSC" "C9808"
+		(property "LCSC" ""
 			(at 248.92 68.58 0)
 			(hide yes)
@@
 			)
 		)
-		(property "Value" "100n"
+		(property "Value" "100nF"
 			(at 33.02 163.83 0)
 			(show_name no)
@@
 			)
 		)
-		(property "LCSC" "C49678"
+		(property "LCSC" ""
 			(at 29.21 162.56 0)
 			(hide yes)
@@
 			)
 		)
-		(property "Value" "100n"
+		(property "Value" "100nF"
 			(at 33.02 129.54 0)
 			(show_name no)
@@
 			)
 		)
-		(property "LCSC" "C49678"
+		(property "LCSC" ""
 			(at 29.21 128.27 0)
 			(hide yes)
@@
 			)
 		)
-		(property "LCSC" "C9808"
+		(property "LCSC" ""
 			(at 203.2 52.07 0)
 			(hide yes)
@@
 			)
 		)
-		(property "LCSC" "C17630"
+		(property "LCSC" ""
 			(at 43.18 158.75 0)
 			(hide yes)
@@
 			)
 		)
-		(property "LCSC" "C9808"
+		(property "LCSC" ""
 			(at 187.96 52.07 0)
 			(hide yes)
@@
 			)
 		)
-		(property "Value" "100n"
+		(property "Value" "100nF"
 			(at 45.72 129.54 0)
 			(show_name no)
@@
 			)
 		)
-		(property "LCSC" "C49678"
+		(property "LCSC" ""
 			(at 41.91 128.27 0)
 			(hide yes)
@@
 			)
 		)
-		(property "LCSC" "C9808"
+		(property "LCSC" ""
 			(at 218.44 52.07 0)
 			(hide yes)
@@
 			)
 		)
-		(property "LCSC" "C9808"
+		(property "LCSC" ""
 			(at 233.68 52.07 0)
 			(hide yes)
@@
 			)
 		)
-		(property "LCSC" "C9808"
+		(property "LCSC" ""
 			(at 218.44 35.56 0)
 			(hide yes)
@@
 			)
 		)
-		(property "LCSC" "C9808"
+		(property "LCSC" ""
 			(at 203.2 68.58 0)
 			(hide yes)
@@
 			)
 		)
-		(property "Value" "10K"
+		(property "Value" "10k"
 			(at 48.26 182.88 90)
 			(show_name no)
@@
 			)
 		)
-		(property "LCSC" "C17414"
+		(property "LCSC" ""
 			(at 48.26 186.69 0)
 			(hide yes)
@@
 			)
 		)
-		(property "LCSC" "C9808"
+		(property "LCSC" ""
 			(at 233.68 35.56 0)
 			(hide yes)
@@
 			)
 		)
-		(property "LCSC" "C9808"
+		(property "LCSC" ""
 			(at 248.92 52.07 0)
 			(hide yes)
@@
 			)
 		)
-		(property "LCSC" "C9808"
+		(property "LCSC" ""
 			(at 187.96 68.58 0)
 			(hide yes)
@@
 			)
 		)
-		(property "LCSC" "C9808"
+		(property "LCSC" ""
 			(at 233.68 68.58 0)
 			(hide yes)
@@
 			)
 		)
-		(property "LCSC" "C27834"
+		(property "LCSC" ""
 			(at 68.58 78.74 0)
 			(hide yes)
@@
 			)
 		)
-		(property "LCSC" "C9808"
+		(property "LCSC" ""
 			(at 203.2 35.56 0)
 			(hide yes)
@@
 			)
 		)
-		(property "LCSC" "C9808"
+		(property "LCSC" ""
 			(at 218.44 68.58 0)
 			(hide yes)
@@
 			)
 		)
-		(property "LCSC" "C9808"
+		(property "LCSC" ""
 			(at 187.96 35.56 0)
 			(hide yes)
