File: pcb/keyboard-ch552-48-lpr.kicad_pcb (KiCad board)
At the start: 2 copper layers, 224.6 x 73.2 mm, 112 parts, among them J1 USB_C_Receptacle_USB2.0, SW1 SW_SPST, SW2 SW_SPST, U1 CH552T

Commit message: pcb: tidy values in ch552-48-lpr
Parts:
- C1, C2, C3: value 100n -> 100nF
- J1: value USB_C_Receptacle_USB2.0 -> USB Type-C Female 16P
- R2: value 10K -> 10k
