File: pcb/keyboard-pykey40-hsrgb.kicad_pcb (KiCad board)
At the start: 2 copper layers, 227 x 77 mm, 244 parts, among them J1 USB_C_Receptacle_USB2.0, J2 Conn_01x03, Q1 Q_NMOS_GSD, U1 RP2040, U2 W25Q128JVS, U3 USBLC6-2SC6, U4 AMS1117-3.3, Y1 12MHz

Commit message: pcb: tidy values in pykey40-hsrgb
Parts:
- C1, C14, C2, C3, C4, C5, C6, C7, C8, C9, C_1_1, C_1_10, C_1_11, C_1_12, C_1_2, C_1_3, C_1_4, C_1_5, C_1_6, C_1_7, C_1_8, C_1_9, C_2_1, C_2_10, C_2_11, C_2_12, C_2_2, C_2_3, C_2_4, C_2_5, C_2_6, C_2_7, C_2_8, C_2_9, C_3_1, C_3_10, C_3_11, C_3_12, C_3_2, C_3_3, C_3_4, C_3_5, C_3_6, C_3_7, C_3_8, C_3_9, C_4_1, C_4_10, C_4_11, C_4_12, C_4_2, C_4_3, C_4_4, C_4_5, C_4_6, C_4_7, C_4_8, C_4_9, C_BL_1, C_BL_2, C_BL_3, C_BL_4: value 100n -> 100nF
- C10, C11: value 1u -> 1uF
- C12, C13: value 22p -> 22pF
- C15, C16: value 22u -> 22uF
- J1: value USB_C_Receptacle_USB2.0 -> USB Type-C Female 16P
- R3, R4: value 22 -> 22R
