File: pcb/keyboard-pykey40-hsrgb.kicad_sch (KiCad schematic)
At the start: 137 parts, among them J1 USB_C_Receptacle_USB2.0, J2 Conn_01x03, U1 RP2040, U2 W25Q128JVS, U3 USBLC6-2SC6, U4 AMS1117-3.3, Y1 12MHz

Commit message: pcb: tidy values in pykey40-hsrgb
Parts:
- C1, C14, C2, C3, C4, C5, C6, C7, C8, C9: value 100n -> 100nF
- C10, C11: value 1u -> 1uF
- C12, C13: value 22p -> 22pF
- C15, C16: value 22u -> 22uF
- J1: value USB_C_Receptacle_USB2.0 -> USB Type-C Female 16P
- R3, R4: value 22 -> 22R
Changed lines of the file:
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@@
 			)
 		)
-		(property "Value" "USB_C_Receptacle_USB2.0"
+		(property "Value" "USB Type-C Female 16P"
 			(at 31.9278 116.9416 0)
 			(show_name no)
@@
 			)
 		)
-		(property "Value" "100n"
+		(property "Value" "100nF"
 			(at 200.787 127.381 0)
 			(show_name no)
@@
 			)
 		)
-		(property "Value" "22"
+		(property "Value" "22R"
 			(at 382.524 141.3256 90)
 			(show_name no)
@@
 			)
 		)
-		(property "Value" "22"
+		(property "Value" "22R"
 			(at 382.524 151.13 90)
 			(show_name no)
@@
 			)
 		)
-		(property "Value" "100n"
+		(property "Value" "100nF"
 			(at 343.535 117.475 0)
 			(show_name no)
@@
 			)
 		)
-		(property "Value" "100n"
+		(property "Value" "100nF"
 			(at 353.695 117.475 0)
 			(show_name no)
@@
 			)
 		)
-		(property "Value" "100n"
+		(property "Value" "100nF"
 			(at 362.585 117.475 0)
 			(show_name no)
@@
 			)
 		)
-		(property "Value" "100n"
+		(property "Value" "100nF"
 			(at 371.475 117.475 0)
 			(show_name no)
@@
 			)
 		)
-		(property "Value" "100n"
+		(property "Value" "100nF"
 			(at 380.365 117.475 0)
 			(show_name no)
@@
 			)
 		)
-		(property "Value" "100n"
+		(property "Value" "100nF"
 			(at 390.525 117.475 0)
 			(show_name no)
@@
 			)
 		)
-		(property "Value" "100n"
+		(property "Value" "100nF"
 			(at 399.415 117.475 0)
 			(show_name no)
@@
 			)
 		)
-		(property "Value" "100n"
+		(property "Value" "100nF"
 			(at 320.675 117.475 0)
 			(show_name no)
@@
 			)
 		)
-		(property "Value" "100n"
+		(property "Value" "100nF"
 			(at 309.245 117.475 0)
 			(show_name no)
@@
 			)
 		)
-		(property "Value" "1u"
+		(property "Value" "1uF"
 			(at 320.675 131.445 0)
 			(show_name no)
@@
 			)
 		)
-		(property "Value" "1u"
+		(property "Value" "1uF"
 			(at 368.935 131.445 0)
 			(show_name no)
@@
 			)
 		)
-		(property "Value" "22p"
+		(property "Value" "22pF"
 			(at 272.034 192.2526 90)
 			(show_name no)
@@
 			)
 		)
-		(property "Value" "22p"
+		(property "Value" "22pF"
 			(at 272.034 183.3626 90)
 			(show_name no)
@@
 			)
 		)
-		(property "Value" "22u"
+		(property "Value" "22uF"
 			(at 78.613 194.437 0)
 			(show_name no)
@@
 			)
 		)
-		(property "Value" "22u"
+		(property "Value" "22uF"
 			(at 46.863 193.167 0)
 			(show_name no)
