File: pcb/keyboard-pykey40-lite.kicad_sch (KiCad schematic)
At the start: 135 parts, among them J1 USB_C_Receptacle_USB2.0, J2 Conn_01x03, U1 RP2040, U2 W25Q128JVS, U3 USBLC6-2SC6, U4 AMS1117-3.3, Y1 12MHz

Commit message: pcb: tidy values in pykey40-lite
Parts:
- C1, C14, C2, C3, C4, C5, C6, C7, C8, C9: value 100n -> 100nF
- C10, C11: value 1u -> 1uF
- C12, C13: value 22p -> 22pF
- C15, C16: value 22u -> 22uF
- J1: value USB_C_Receptacle_USB2.0 -> USB Type-C Female 16P
- R3, R4: value 22 -> 22R
Changed lines of the file:
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@@
 			)
 		)
-		(property "Value" "USB_C_Receptacle_USB2.0"
+		(property "Value" "USB Type-C Female 16P"
 			(at 31.9278 117.4496 0)
 			(show_name no)
@@
 			)
 		)
-		(property "Value" "100n"
+		(property "Value" "100nF"
 			(at 178.181 128.143 0)
 			(show_name no)
@@
 			)
 		)
-		(property "Value" "22"
+		(property "Value" "22R"
 			(at 295.91 151.13 90)
 			(show_name no)
@@
 			)
 		)
-		(property "Value" "22"
+		(property "Value" "22R"
 			(at 295.91 153.67 90)
 			(show_name no)
@@
 			)
 		)
-		(property "Value" "100n"
+		(property "Value" "100nF"
 			(at 256.921 124.333 0)
 			(show_name no)
@@
 			)
 		)
-		(property "Value" "100n"
+		(property "Value" "100nF"
 			(at 267.081 124.333 0)
 			(show_name no)
@@
 			)
 		)
-		(property "Value" "100n"
+		(property "Value" "100nF"
 			(at 275.971 124.333 0)
 			(show_name no)
@@
 			)
 		)
-		(property "Value" "100n"
+		(property "Value" "100nF"
 			(at 284.861 124.333 0)
 			(show_name no)
@@
 			)
 		)
-		(property "Value" "100n"
+		(property "Value" "100nF"
 			(at 293.751 124.333 0)
 			(show_name no)
@@
 			)
 		)
-		(property "Value" "100n"
+		(property "Value" "100nF"
 			(at 303.911 124.333 0)
 			(show_name no)
@@
 			)
 		)
-		(property "Value" "100n"
+		(property "Value" "100nF"
 			(at 312.801 124.333 0)
 			(show_name no)
@@
 			)
 		)
-		(property "Value" "100n"
+		(property "Value" "100nF"
 			(at 234.061 124.333 0)
 			(show_name no)
@@
 			)
 		)
-		(property "Value" "100n"
+		(property "Value" "100nF"
 			(at 222.631 124.333 0)
 			(show_name no)
@@
 			)
 		)
-		(property "Value" "1u"
+		(property "Value" "1uF"
 			(at 226.06 138.43 0)
 			(show_name no)
@@
 			)
 		)
-		(property "Value" "1u"
+		(property "Value" "1uF"
 			(at 282.321 138.303 0)
 			(show_name no)
@@
 			)
 		)
-		(property "Value" "22p"
+		(property "Value" "22pF"
 			(at 185.42 199.1106 90)
 			(show_name no)
@@
 			)
 		)
-		(property "Value" "22p"
+		(property "Value" "22pF"
 			(at 185.42 190.2206 90)
 			(show_name no)
@@
 			)
 		)
-		(property "Value" "22u"
+		(property "Value" "22uF"
 			(at 85.471 197.993 0)
 			(show_name no)
@@
 			)
 		)
-		(property "Value" "22u"
+		(property "Value" "22uF"
 			(at 53.721 196.723 0)
 			(show_name no)
