File: pcb/keyboard-x2-lumberjack-arm-hsrgb.kicad_pcb (KiCad board)
At the start: 2 copper layers, 285 x 94.2 mm, 276 parts, among them J1 16-pin USB-C Connector SMD, U1 STM32F103 Bluepill, or MiniF4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, U2 SN74LVC1T45DBV

Commit message: pcb: tidy values in lumberjack-arm-hsrgb
Parts:
- R1, R2: value 5.1K -> 5.1k
