File: pcb/keyboard-x2-lumberjack-arm-hsrgb.kicad_sch (KiCad schematic)
At the start: 13 parts, among them J1 16-pin USB-C Connector SMD, U1 STM32F103 Bluepill, or MiniF4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, U2 SN74LVC1T45DBV

Commit message: pcb: upgrade to kicad 10: keyboard-x2-lumberjack-arm-hsrgb
Parts:
- H5: value ~ -> (none)

Commit message: pcb: tidy values in lumberjack-arm-hsrgb
Parts:
- R1, R2: value 5.1K -> 5.1k
Changed lines of the file:
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@@
 			)
 		)
-		(property "Value" "5.1K"
+		(property "Value" "5.1k"
 			(at 56.388 112.903 0)
 			(show_name no)
@@
 			)
 		)
-		(property "Value" "5.1K"
+		(property "Value" "5.1k"
 			(at 66.548 112.903 0)
 			(show_name no)
