File: pcb/keyboard-wabble-60.kicad_pcb (KiCad board)
At the start: 2 copper layers, 285 x 94.2 mm, 151 parts, among them J1 16-pin USB-C Connector SMD, J2 Battery, J3 2-pin PH2.0 JST, J4 2-pin PH2.0 JST, J5 Conn_01x03_Socket, J6 Conn_01x02_Socket, Q2 BSS138, SW1 SS-12F44, U1 WeAct WCH BLE CoreBoard, U2 TP4054

Commit message: pcb: tidy values in wabble-60
Parts:
- R1, R2: value 5.1K -> 5.1k
- R3: value 22K -> 22k
- R4: value 10K -> 10k
