File: pcb/keyboard-wabble-60.kicad_sch (KiCad schematic)
At the start: 149 parts, among them J1 16-pin USB-C Connector SMD, J2 Battery, J3 2-pin PH2.0 JST, J4 2-pin PH2.0 JST, J5 Conn_01x03_Socket, J6 Conn_01x02_Socket, Q2 BSS138, SW1 SS-12F44, U1 WeAct WCH BLE CoreBoard, U2 TP4054

Commit message: pcb: upgrade to kicad 10: keyboard-wabble-60
Parts:
- H5: value ~ -> (none)

Commit message: pcb: tidy values in wabble-60
Parts:
- R1, R2: value 5.1K -> 5.1k
- R3: value 22K -> 22k
- R4: value 10K -> 10k
Changed lines of the file:
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@@
 			)
 		)
-		(property "Value" "5.1K"
+		(property "Value" "5.1k"
 			(at 56.388 81.153 0)
 			(show_name no)
@@
 			)
 		)
-		(property "Value" "5.1K"
+		(property "Value" "5.1k"
 			(at 56.388 98.933 0)
 			(show_name no)
@@
 			)
 		)
-		(property "Value" "22K"
+		(property "Value" "22k"
 			(at 87.63 177.8 90)
 			(show_name no)
@@
 			)
 		)
-		(property "Value" "10K"
+		(property "Value" "10k"
 			(at 99.06 133.35 0)
 			(show_name no)
