File: pcb/keyboard-ch32x-36-lhs.kicad_pcb (KiCad board)
At the start: 2 copper layers, 100 x 96.5 mm, 57 parts, among them J1 USB Type-C Receptacle 12-pin, J2 PJ-320A, J4 Conn_01x02, J5 Conn_01x03, SW1 SW_SPST, SW2 SW_SPST, U1 CH32X033F8P6

Commit message: pcb: tidy values in ch32x-36
Parts:
- C1, C3: value 100n -> 100nF
- R4: value 10K -> 10k
