File: pcb/keyboard-ch32x-36-lhs.kicad_sch (KiCad schematic)
At the start: 57 parts, among them J1 USB Type-C Receptacle 12-pin, J2 PJ-320A, J4 Conn_01x02, J5 Conn_01x03, SW1 SW_SPST, SW2 SW_SPST, U1 CH32X033F8P6

Commit message: pcb: tidy values in ch32x-36
Parts:
- C1, C3: value 100n -> 100nF; LCSC C28233 -> (none)
- C2: LCSC C1779 -> (none)
- R1, R2: LCSC C27834 -> (none)
- R3: LCSC C17630 -> (none)
- R4: value 10K -> 10k; LCSC C17414 -> (none)
Changed lines of the file:
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@@
 			)
 		)
-		(property "LCSC" "C27834"
+		(property "LCSC" ""
 			(at 64.77 77.47 0)
 			(hide yes)
@@
 			)
 		)
-		(property "LCSC" "C1779"
+		(property "LCSC" ""
 			(at 38.1 123.19 0)
 			(hide yes)
@@
 			)
 		)
-		(property "LCSC" "C17630"
+		(property "LCSC" ""
 			(at 53.34 176.53 0)
 			(hide yes)
@@
 			)
 		)
-		(property "Value" "100n"
+		(property "Value" "100nF"
 			(at 54.61 124.46 0)
 			(show_name no)
@@
 			)
 		)
-		(property "LCSC" "C28233"
+		(property "LCSC" ""
 			(at 50.8 123.19 0)
 			(hide yes)
@@
 			)
 		)
-		(property "Value" "10K"
+		(property "Value" "10k"
 			(at 54.61 148.59 90)
 			(show_name no)
@@
 			)
 		)
-		(property "LCSC" "C17414"
+		(property "LCSC" ""
 			(at 54.61 152.4 0)
 			(hide yes)
@@
 			)
 		)
-		(property "Value" "100n"
+		(property "Value" "100nF"
 			(at 43.18 181.6099 0)
 			(show_name no)
@@
 			)
 		)
-		(property "LCSC" "C28233"
+		(property "LCSC" ""
 			(at 39.37 180.34 0)
 			(hide yes)
@@
 			)
 		)
-		(property "LCSC" "C27834"
+		(property "LCSC" ""
 			(at 74.93 77.47 0)
 			(hide yes)
