File: pcb/keyboard-ch32x-75.kicad_pcb (KiCad board)
At the start: 2 copper layers, 285 x 94.2 mm, 325 parts, among them J1 USB_C_Receptacle_USB2.0, J2 Conn_01x02, J3 Conn_01x04, Q1 AO3400A, SW1 SW_SPST, SW2 SW_SPST, U1 CH32X035C8T6, U2 USBLC6-2SC6

Commit message: pcb: tidy values in ch32x-75
Parts:
- C1, C2: value 100n -> 100nF
- J1: value USB_C_Receptacle_USB2.0 -> USB Type-C Female 16P
- R1, R4, R5, R7: value 10K -> 10k
