File: pcb/keyboard-ch32x-60-improved.kicad_sch (KiCad schematic)
At the start: 157 parts, among them J1 USB Type-C Female 16P, J2 Conn_01x02, J3 Conn_01x04, SW1 SW_SPST, SW2 SW_SPST, U1 CH32X035C8T6, U2 USBLC6-2SC6

Commit message: pcb: update comment
Other:
- note added: "WCH Link interface (CH32X033 only compatible with WCH-LinkE or WCH-LinkW)"
- note removed: "WCH Link interface (CH32X033 only compatible with WCH-LinkE or WCH-LinkW) Using DIO/DCK prevents use of ROW2/ROW6."
Changed lines of the file:
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@@
 		)
 	)
-	(text "WCH Link interface\n(CH32X033 only compatible with WCH-LinkE or WCH-LinkW)\nUsing DIO/DCK prevents use of ROW2/ROW6."
+	(text "WCH Link interface\n(CH32X033 only compatible with WCH-LinkE or WCH-LinkW)"
 		(exclude_from_sim no)
 		(at 14.986 250.698 0)

Commit message: pcb: update comment in schematic
Other:
- note added: "UART For simple printf debugging with UART2."
- note removed: "UART For simple printf debugging with UART2. ("ROW4"/SW_4_x switches can't be used while using UART2)."
Changed lines of the file:
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@@
 		)
 	)
-	(text "UART\nFor simple printf debugging with UART2.\n(\"ROW4\"/SW_4_x switches can't be used\n while using UART2)."
+	(text "UART\nFor simple printf debugging with UART2."
 		(exclude_from_sim no)
 		(at 14.732 230.124 0)
