File: pcb/keyboard-ch32x-75.kicad_sch (KiCad schematic)
At the start: 325 parts, among them J1 USB_C_Receptacle_USB2.0, J2 Conn_01x02, J3 Conn_01x04, Q1 AO3400A, SW1 SW_SPST, SW2 SW_SPST, U1 CH32X035C8T6, U2 USBLC6-2SC6

Commit message: pcb: tidy values in ch32x-75
Parts:
- C1, C2: value 100n -> 100nF; LCSC C28233 -> (none)
- C3: LCSC C1779 -> (none)
- D_1_1, D_1_10, D_1_11, D_1_12, D_1_13, D_1_14, D_1_15, D_1_2, D_1_3, D_1_4, D_1_5, D_1_6, D_1_7, D_1_8, D_1_9, D_2_1, D_2_10, D_2_11, D_2_12, D_2_13, D_2_14, D_2_15, D_2_2, D_2_3, D_2_4, D_2_5, D_2_6, D_2_7, D_2_8, D_2_9, D_3_1, D_3_10, D_3_11, D_3_12, D_3_13, D_3_14, D_3_15, D_3_2, D_3_3, D_3_4, D_3_5, D_3_6, D_3_7, D_3_8, D_3_9, D_4_1, D_4_10, D_4_11, D_4_12, D_4_13, D_4_14, D_4_15, D_4_2, D_4_3, D_4_4, D_4_5, D_4_6, D_4_7, D_4_8, D_4_9, D_5_1, D_5_10, D_5_11, D_5_12, D_5_13, D_5_14, D_5_15, D_5_2, D_5_3, D_5_4, D_5_5, D_5_6, D_5_7, D_5_8, D_5_9: LCSC C9808 -> (none)
- J1: value USB_C_Receptacle_USB2.0 -> USB Type-C Female 16P
- R1, R4, R5, R7: value 10K -> 10k; LCSC C17414 -> (none)
- R2, R3: LCSC C27834 -> (none)
- R6: LCSC C17414 -> (none)

Commit message: pcb: update comment in schematic
Other:
- note added: "UART For simple printf debugging with UART2."
- note added: "WCH Link interface (CH32X033 only compatible with WCH-LinkE or WCH-LinkW)"
- note removed: "UART For simple printf debugging with UART2. ("ROW4"/SW_4_x switches can't be used while using UART2)."
- note removed: "WCH Link interface (CH32X033 only compatible with WCH-LinkE or WCH-LinkW) Using DIO/DCK prevents use of ROW2/ROW6."
Changed lines of the file:
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@@
 		)
 	)
-	(text "WCH Link interface\n(CH32X033 only compatible with WCH-LinkE or WCH-LinkW)\nUsing DIO/DCK prevents use of ROW2/ROW6."
+	(text "WCH Link interface\n(CH32X033 only compatible with WCH-LinkE or WCH-LinkW)"
 		(exclude_from_sim no)
 		(at 14.986 250.698 0)
@@
 		)
 	)
-	(text "UART\nFor simple printf debugging with UART2.\n(\"ROW4\"/SW_4_x switches can't be used\n while using UART2)."
+	(text "UART\nFor simple printf debugging with UART2."
 		(exclude_from_sim no)
 		(at 14.732 230.124 0)
